Commit message: fix(sim): inject roller contact surfaces into generated SDF

File: mobile_base_description/urdf/macros/mecanum_rollers.xacro (robot description, xacro)
@@ -87,9 +87,13 @@
                   friction="${roller_joint_friction}"/>
       </joint>
+      <!--
+        Contact friction and stiffness are NOT set here. mu1/mu2/kp/kd are
+        Gazebo-Classic extension tags that gz sdf -p silently discards during
+        URDF-to-SDF conversion, so authoring them here has no effect on the
+        simulated contact. generate_sim_sdf.py injects a real SDF <surface>
+        into every roller collision instead, and refuses to emit a model
+        whose rollers lack one. Keep that script the single authority.
+      -->
       <gazebo reference="${prefix}${wheel_name}_roller_${index}_link">
-        <mu1>${roller_contact_mu}</mu1>
-        <mu2>${roller_contact_mu}</mu2>
-        <kp>${roller_contact_kp}</kp>
-        <kd>${roller_contact_kd}</kd>
         <selfCollide>false</selfCollide>
       </gazebo>

File: mobile_base_description/urdf/properties.xacro (robot description, xacro)
@@ -23,10 +23,14 @@
   <xacro:property name="roller_joint_friction"
                   value="$(arg roller_joint_friction)"/>
-  <xacro:property name="roller_contact_mu"
-                  value="$(arg roller_contact_mu)"/>
   <xacro:property name="roller_collision_model"
                   value="$(arg roller_collision_model)"/>
-  <xacro:property name="roller_contact_kp" value="100000.0"/>
-  <xacro:property name="roller_contact_kd" value="10.0"/>
+  <!--
+    Contact friction and stiffness (mu, mu2, kp, kd) are intentionally absent
+    here. They cannot be expressed in a URDF that survives gz sdf -p, so they
+    are applied by mobile_base_bringup/scripts/generate_sim_sdf.py when the
+    simulation SDF is produced. The roller_contact_mu xacro argument is still
+    accepted so callers can pass it uniformly, but it shapes the generated
+    SDF rather than this description.
+  -->
   <!-- wheelbase is front-to-rear wheel-center spacing; wheel_separation is track width. -->
   <xacro:property name="wheelbase" value="0.150"/>
