Commit message: feat(sim): add husarion_cylinder anisotropic wheel contact model

File: mobile_base_description/urdf/macros/mecanum_wheels.xacro (robot description, xacro)
@@ -15,4 +15,19 @@
         <material name="wheel_orange"/>
       </visual>
+      <!--
+        The explicit-roller models put every ground contact on the passive
+        roller links and leave the driven hub without collision. The
+        husarion_cylinder model instead gives the hub one cylinder and
+        reproduces the mecanum effect with a direction-dependent friction
+        cone: 4 contacts instead of 360.
+      -->
+      <xacro:unless value="${explicit_rollers}">
+        <collision name="wheel_collision">
+          <origin xyz="0 0 0" rpy="${pi / 2.0} 0 0"/>
+          <geometry>
+            <cylinder radius="${wheel_radius}" length="${wheel_width}"/>
+          </geometry>
+        </collision>
+      </xacro:unless>
       <xacro:cylinder_inertial mass="${wheel_hub_mass}"
                                radius="${roller_center_radius}"
@@ -26,16 +41,28 @@
       <origin xyz="${x} ${y} ${z}" rpy="0 0 0"/>
       <axis xyz="0 1 0"/>
-      <dynamics damping="0.05" friction="0.01"/>
+      <dynamics damping="${wheel_joint_damping}"
+                friction="${wheel_joint_friction}"/>
       <limit effort="8.0" velocity="25.0"/>
     </joint>
+    <!--
+      No contact parameters here on purpose. gz sdf -p discards every friction
+      form written inside a gazebo reference block: both the Gazebo-Classic
+      mu1/kp tags and nested SDF collision/surface. Anything set here would
+      silently do nothing in this pipeline. Husarion can author friction in
+      their xacro because they spawn the URDF directly; this repo pre-converts
+      to SDF, so generate_sim_sdf.py injects the wheel surface (mu, mu2,
+      slip1, and the handed fdir1) after conversion instead.
+    -->
     <gazebo reference="${prefix}${name}_wheel_link">
       <selfCollide>false</selfCollide>
     </gazebo>
-    <xacro:mecanum_roller_ring
-      prefix="${prefix}"
-      wheel_name="${name}"
-      roller_handedness="${roller_handedness}"
-      roller_phase="${roller_phase}"
-      roller_axial_offset="${roller_axial_offset}"/>
+    <xacro:if value="${explicit_rollers}">
+      <xacro:mecanum_roller_ring
+        prefix="${prefix}"
+        wheel_name="${name}"
+        roller_handedness="${roller_handedness}"
+        roller_phase="${roller_phase}"
+        roller_axial_offset="${roller_axial_offset}"/>
+    </xacro:if>
   </xacro:macro>
 </robot>

File: mobile_base_description/urdf/mobile_base.ros2_control.xacro (robot description, xacro)
@@ -37,8 +37,14 @@
       <xacro:wheel_interface joint_name="rear_right_wheel_joint"/>
       <xacro:wheel_interface joint_name="rear_left_wheel_joint"/>
-      <xacro:roller_state_interfaces wheel_name="front_left"/>
-      <xacro:roller_state_interfaces wheel_name="front_right"/>
-      <xacro:roller_state_interfaces wheel_name="rear_right"/>
-      <xacro:roller_state_interfaces wheel_name="rear_left"/>
+      <!--
+        Every joint named in a ros2_control block must exist in the URDF, so
+        the roller interfaces are emitted only when the roller links are.
+      -->
+      <xacro:if value="${explicit_rollers}">
+        <xacro:roller_state_interfaces wheel_name="front_left"/>
+        <xacro:roller_state_interfaces wheel_name="front_right"/>
+        <xacro:roller_state_interfaces wheel_name="rear_right"/>
+        <xacro:roller_state_interfaces wheel_name="rear_left"/>
+      </xacro:if>
     </ros2_control>
   </xacro:macro>

File: mobile_base_description/urdf/mobile_base.urdf.xacro (robot description, xacro)
@@ -8,4 +8,9 @@
   <xacro:arg name="roller_contact_mu" default="1.0"/>
   <xacro:arg name="roller_collision_model" default="barrel"/>
+  <!-- husarion_cylinder anisotropic wheel contact; ignored by other models. -->
+  <xacro:arg name="wheel_contact_mu" default="0.8"/>
+  <xacro:arg name="wheel_contact_mu2" default="0.2"/>
+  <xacro:arg name="wheel_contact_slip1" default="0.0"/>
+  <xacro:arg name="wheel_contact_slip2" default="0.0"/>
   <xacro:arg name="front_left_roller_phase" default="0.22193969"/>
   <xacro:arg name="front_right_roller_phase" default="0.48030419"/>

File: mobile_base_description/urdf/properties.xacro (robot description, xacro)
@@ -17,6 +17,4 @@
   <xacro:property name="roller_inclination" value="${pi / 4.0}"/>
   <xacro:property name="roller_mass" value="${wheel_mass * 0.03}"/>
-  <xacro:property name="wheel_hub_mass"
-                  value="${wheel_mass - roller_count * roller_mass}"/>
   <xacro:property name="roller_joint_damping"
                   value="$(arg roller_joint_damping)"/>
@@ -25,4 +23,37 @@
   <xacro:property name="roller_collision_model"
                   value="$(arg roller_collision_model)"/>
+  <!--
+    husarion_cylinder emits no roller links at all, so the hub must carry the
+    whole wheel mass. The explicit-roller models leave the roller ring holding
+    its share. Total wheel mass is 0.12 kg either way.
+  -->
+  <xacro:property name="explicit_rollers"
+                  value="${roller_collision_model != 'husarion_cylinder'}"/>
+  <xacro:property name="wheel_hub_mass"
+                  value="${wheel_mass - roller_count * roller_mass
+                           if explicit_rollers else wheel_mass}"/>
+  <!--
+    Anisotropic wheel contact, used only by husarion_cylinder. A mecanum roller
+    rolls across its own axis and grips along it, so mu acts along fdir1 (the
+    roller axis) and mu2 across it. Values follow the shipping Husarion ROSbot
+    XL configuration; slip1 supplies the tangential compliance without which
+    the single-cylinder contact oscillates instead of translating.
+  -->
+  <!--
+    Driven-joint resistance. With explicit rollers the roller ring carries the
+    sliding and these values are part of the existing calibration, so they are
+    left alone. husarion_cylinder has no rollers, so every bit of joint
+    resistance runs through the wheel joint; the shipping ROSbot XL uses
+    0.001/0.001 there, against 0.05/0.01 here, and the heavier damping shows up
+    as wheel-tracking error.
+  -->
+  <xacro:property name="wheel_joint_damping"
+                  value="${0.05 if explicit_rollers else 0.001}"/>
+  <xacro:property name="wheel_joint_friction"
+                  value="${0.01 if explicit_rollers else 0.001}"/>
+  <xacro:property name="wheel_contact_mu" value="$(arg wheel_contact_mu)"/>
+  <xacro:property name="wheel_contact_mu2" value="$(arg wheel_contact_mu2)"/>
+  <xacro:property name="wheel_contact_slip1" value="$(arg wheel_contact_slip1)"/>
+  <xacro:property name="wheel_contact_slip2" value="$(arg wheel_contact_slip2)"/>
   <!--
     Contact friction and stiffness (mu, mu2, kp, kd) are intentionally absent
