Commit message: fix(mecanum): calibrate physical roller contact geometry

File: mobile_base_description/urdf/base.xacro (robot description, xacro)
@@ -8,5 +8,5 @@
                           z="${wheel_z}" parent="base_link"
                           roller_handedness="-1"
-                          roller_phase="0.22193969"
+                          roller_phase="$(arg front_left_roller_phase)"
                           roller_axial_offset="-0.00059729"
                           mesh="mecanum_wheel_FL.stl"
@@ -17,5 +17,5 @@
                           z="${wheel_z}" parent="base_link"
                           roller_handedness="1"
-                          roller_phase="0.48030419"
+                          roller_phase="$(arg front_right_roller_phase)"
                           roller_axial_offset="0.00059729"
                           mesh="mecanum_wheel_FR.stl"
@@ -26,5 +26,5 @@
                           z="${wheel_z}" parent="base_link"
                           roller_handedness="-1"
-                          roller_phase="0.19668582"
+                          roller_phase="$(arg rear_right_roller_phase)"
                           roller_axial_offset="0.00059729"
                           mesh="mecanum_wheel_RR.stl"
@@ -35,5 +35,5 @@
                           z="${wheel_z}" parent="base_link"
                           roller_handedness="1"
-                          roller_phase="0.24790784"
+                          roller_phase="$(arg rear_left_roller_phase)"
                           roller_axial_offset="-0.00059729"
                           mesh="mecanum_wheel_RL.stl"

File: mobile_base_description/urdf/macros/mecanum_rollers.xacro (robot description, xacro)
@@ -26,10 +26,49 @@
                       value="${atan2(sqrt(axis_dx * axis_dx + axis_dy * axis_dy), axis_dz)}"/>
       <link name="${prefix}${wheel_name}_roller_${index}_link">
-        <collision>
-          <origin xyz="0 0 0" rpy="0 0 0"/>
-          <geometry>
-            <cylinder radius="${roller_radius}" length="${roller_length}"/>
-          </geometry>
-        </collision>
+        <xacro:if value="${roller_collision_model == 'cylinder'}">
+          <collision name="cylinder_collision">
+            <origin xyz="0 0 0" rpy="0 0 0"/>
+            <geometry>
+              <cylinder radius="${roller_radius}" length="${roller_length}"/>
+            </geometry>
+          </collision>
+        </xacro:if>
+        <xacro:if value="${roller_collision_model == 'barrel'}">
+          <collision name="barrel_center_collision">
+            <geometry><sphere radius="0.00569443"/></geometry>
+          </collision>
+          <collision name="barrel_negative_3mm_collision">
+            <origin xyz="0 0 -0.003" rpy="0 0 0"/>
+            <geometry><sphere radius="0.00558"/></geometry>
+          </collision>
+          <collision name="barrel_positive_3mm_collision">
+            <origin xyz="0 0 0.003" rpy="0 0 0"/>
+            <geometry><sphere radius="0.00558"/></geometry>
+          </collision>
+          <collision name="barrel_negative_5p8mm_collision">
+            <origin xyz="0 0 -0.0058" rpy="0 0 0"/>
+            <geometry><sphere radius="0.00526"/></geometry>
+          </collision>
+          <collision name="barrel_positive_5p8mm_collision">
+            <origin xyz="0 0 0.0058" rpy="0 0 0"/>
+            <geometry><sphere radius="0.00526"/></geometry>
+          </collision>
+          <collision name="barrel_negative_8p2mm_collision">
+            <origin xyz="0 0 -0.0082" rpy="0 0 0"/>
+            <geometry><sphere radius="0.0048"/></geometry>
+          </collision>
+          <collision name="barrel_positive_8p2mm_collision">
+            <origin xyz="0 0 0.0082" rpy="0 0 0"/>
+            <geometry><sphere radius="0.0048"/></geometry>
+          </collision>
+          <collision name="barrel_negative_10p8mm_collision">
+            <origin xyz="0 0 -0.0108" rpy="0 0 0"/>
+            <geometry><sphere radius="0.00405"/></geometry>
+          </collision>
+          <collision name="barrel_positive_10p8mm_collision">
+            <origin xyz="0 0 0.0108" rpy="0 0 0"/>
+            <geometry><sphere radius="0.00405"/></geometry>
+          </collision>
+        </xacro:if>
         <xacro:cylinder_inertial mass="${roller_mass}"
                                  radius="${roller_radius}"

File: mobile_base_description/urdf/mobile_base.urdf.xacro (robot description, xacro)
@@ -4,4 +4,12 @@
   <xacro:arg name="use_gazebo" default="false"/>
   <xacro:arg name="controllers_file" default=""/>
+  <xacro:arg name="roller_joint_damping" default="0.0"/>
+  <xacro:arg name="roller_joint_friction" default="0.0"/>
+  <xacro:arg name="roller_contact_mu" default="0.8"/>
+  <xacro:arg name="roller_collision_model" default="barrel"/>
+  <xacro:arg name="front_left_roller_phase" default="0.22193969"/>
+  <xacro:arg name="front_right_roller_phase" default="0.48030419"/>
+  <xacro:arg name="rear_right_roller_phase" default="0.19668582"/>
+  <xacro:arg name="rear_left_roller_phase" default="0.24790784"/>
   <xacro:include filename="materials.xacro"/>
   <xacro:include filename="inertials.xacro"/>

File: mobile_base_description/urdf/properties.xacro (robot description, xacro)
@@ -19,7 +19,12 @@
   <xacro:property name="wheel_hub_mass"
                   value="${wheel_mass - roller_count * roller_mass}"/>
-  <xacro:property name="roller_joint_damping" value="0.001"/>
-  <xacro:property name="roller_joint_friction" value="0.00005"/>
-  <xacro:property name="roller_contact_mu" value="0.8"/>
+  <xacro:property name="roller_joint_damping"
+                  value="$(arg roller_joint_damping)"/>
+  <xacro:property name="roller_joint_friction"
+                  value="$(arg roller_joint_friction)"/>
+  <xacro:property name="roller_contact_mu"
+                  value="$(arg roller_contact_mu)"/>
+  <xacro:property name="roller_collision_model"
+                  value="$(arg roller_collision_model)"/>
   <xacro:property name="roller_contact_kp" value="100000.0"/>
   <xacro:property name="roller_contact_kd" value="10.0"/>

Commit message: refactor(mecanum): make anisotropic wheel contact canonical

File: mobile_base_description/urdf/base.xacro (robot description, xacro)
@@ -7,7 +7,4 @@
                           x="${wheelbase / 2.0}" y="${wheel_separation / 2.0}"
                           z="${wheel_z}" parent="base_link"
-                          roller_handedness="-1"
-                          roller_phase="$(arg front_left_roller_phase)"
-                          roller_axial_offset="-0.00059729"
                           mesh="mecanum_wheel_FL.stl"
                           visual_xyz="0.105356784 0.000987069 0.084068176"
@@ -16,7 +13,4 @@
                           x="${wheelbase / 2.0}" y="${-wheel_separation / 2.0}"
                           z="${wheel_z}" parent="base_link"
-                          roller_handedness="1"
-                          roller_phase="$(arg front_right_roller_phase)"
-                          roller_axial_offset="0.00059729"
                           mesh="mecanum_wheel_FR.stl"
                           visual_xyz="0.050182544 0.126865288 0.125047948"
@@ -25,7 +19,4 @@
                           x="${-wheelbase / 2.0}" y="${-wheel_separation / 2.0}"
                           z="${wheel_z}" parent="base_link"
-                          roller_handedness="-1"
-                          roller_phase="$(arg rear_right_roller_phase)"
-                          roller_axial_offset="0.00059729"
                           mesh="mecanum_wheel_RR.stl"
                           visual_xyz="-0.030863306 0.126451466 0.020233040"
@@ -34,7 +25,4 @@
                           x="${-wheelbase / 2.0}" y="${wheel_separation / 2.0}"
                           z="${wheel_z}" parent="base_link"
-                          roller_handedness="1"
-                          roller_phase="$(arg rear_left_roller_phase)"
-                          roller_axial_offset="-0.00059729"
                           mesh="mecanum_wheel_RL.stl"
                           visual_xyz="-0.032786922 0.001235564 0.016969848"

File: mobile_base_description/urdf/macros/mecanum_wheels.xacro (robot description, xacro)
@@ -3,5 +3,4 @@
   <xacro:macro name="mecanum_wheel"
                params="prefix name parent x y z mesh visual_xyz
-                       roller_handedness roller_phase roller_axial_offset
                        visual_rpy">
     <link name="${prefix}${name}_wheel_link">
@@ -15,21 +14,12 @@
         <material name="wheel_orange"/>
       </visual>
-      <!--
-        The explicit-roller models put every ground contact on the passive
-        roller links and leave the driven hub without collision. The
-        husarion_cylinder model instead gives the hub one cylinder and
-        reproduces the mecanum effect with a direction-dependent friction
-        cone: 4 contacts instead of 360.
-      -->
-      <xacro:unless value="${explicit_rollers}">
-        <collision name="wheel_collision">
-          <origin xyz="0 0 0" rpy="${pi / 2.0} 0 0"/>
-          <geometry>
-            <cylinder radius="${wheel_radius}" length="${wheel_width}"/>
-          </geometry>
-        </collision>
-      </xacro:unless>
-      <xacro:cylinder_inertial mass="${wheel_hub_mass}"
-                               radius="${roller_center_radius}"
+      <collision name="wheel_collision">
+        <origin xyz="0 0 0" rpy="${pi / 2.0} 0 0"/>
+        <geometry>
+          <cylinder radius="${wheel_radius}" length="${wheel_width}"/>
+        </geometry>
+      </collision>
+      <xacro:cylinder_inertial mass="${wheel_mass}"
+                               radius="${wheel_inertial_radius}"
                                length="${wheel_width}">
         <origin xyz="0 0 0" rpy="${pi / 2.0} 0 0"/>
@@ -46,23 +36,11 @@
     </joint>
     <!--
-      No contact parameters here on purpose. gz sdf -p discards every friction
-      form written inside a gazebo reference block: both the Gazebo-Classic
-      mu1/kp tags and nested SDF collision/surface. Anything set here would
-      silently do nothing in this pipeline. Husarion can author friction in
-      their xacro because they spawn the URDF directly; this repo pre-converts
-      to SDF, so generate_sim_sdf.py injects the wheel surface (mu, mu2,
-      slip1, and the handed fdir1) after conversion instead.
+      No contact parameters are authored here because gz sdf -p discards the
+      relevant URDF extension tags. generate_sim_sdf.py injects the canonical
+      anisotropic wheel surface after conversion.
     -->
     <gazebo reference="${prefix}${name}_wheel_link">
       <selfCollide>false</selfCollide>
     </gazebo>
-    <xacro:if value="${explicit_rollers}">
-      <xacro:mecanum_roller_ring
-        prefix="${prefix}"
-        wheel_name="${name}"
-        roller_handedness="${roller_handedness}"
-        roller_phase="${roller_phase}"
-        roller_axial_offset="${roller_axial_offset}"/>
-    </xacro:if>
   </xacro:macro>
 </robot>

File: mobile_base_description/urdf/mobile_base.ros2_control.xacro (robot description, xacro)
@@ -22,29 +22,8 @@
         </joint>
       </xacro:macro>
-      <xacro:macro name="roller_state_interfaces"
-                   params="wheel_name index:=0">
-        <xacro:if value="${index &lt; roller_count}">
-          <joint name="${prefix}${wheel_name}_roller_${index}_joint">
-            <state_interface name="position"/>
-            <state_interface name="velocity"/>
-          </joint>
-          <xacro:roller_state_interfaces wheel_name="${wheel_name}"
-                                         index="${index + 1}"/>
-        </xacro:if>
-      </xacro:macro>
       <xacro:wheel_interface joint_name="front_left_wheel_joint"/>
       <xacro:wheel_interface joint_name="front_right_wheel_joint"/>
       <xacro:wheel_interface joint_name="rear_right_wheel_joint"/>
       <xacro:wheel_interface joint_name="rear_left_wheel_joint"/>
-      <!--
-        Every joint named in a ros2_control block must exist in the URDF, so
-        the roller interfaces are emitted only when the roller links are.
-      -->
-      <xacro:if value="${explicit_rollers}">
-        <xacro:roller_state_interfaces wheel_name="front_left"/>
-        <xacro:roller_state_interfaces wheel_name="front_right"/>
-        <xacro:roller_state_interfaces wheel_name="rear_right"/>
-        <xacro:roller_state_interfaces wheel_name="rear_left"/>
-      </xacro:if>
     </ros2_control>
   </xacro:macro>

File: mobile_base_description/urdf/mobile_base.urdf.xacro (robot description, xacro)
@@ -4,22 +4,8 @@
   <xacro:arg name="use_gazebo" default="false"/>
   <xacro:arg name="controllers_file" default=""/>
-  <xacro:arg name="roller_joint_damping" default="0.0"/>
-  <xacro:arg name="roller_joint_friction" default="0.0"/>
-  <xacro:arg name="roller_contact_mu" default="1.0"/>
-  <xacro:arg name="roller_collision_model" default="barrel"/>
-  <!-- husarion_cylinder anisotropic wheel contact; ignored by other models. -->
-  <xacro:arg name="wheel_contact_mu" default="0.8"/>
-  <xacro:arg name="wheel_contact_mu2" default="0.2"/>
-  <xacro:arg name="wheel_contact_slip1" default="0.0"/>
-  <xacro:arg name="wheel_contact_slip2" default="0.0"/>
-  <xacro:arg name="front_left_roller_phase" default="0.22193969"/>
-  <xacro:arg name="front_right_roller_phase" default="0.48030419"/>
-  <xacro:arg name="rear_right_roller_phase" default="0.19668582"/>
-  <xacro:arg name="rear_left_roller_phase" default="0.24790784"/>
   <xacro:include filename="materials.xacro"/>
   <xacro:include filename="inertials.xacro"/>
   <xacro:include filename="properties.xacro"/>
   <xacro:include filename="chassis.xacro"/>
-  <xacro:include filename="macros/mecanum_rollers.xacro"/>
   <xacro:include filename="macros/mecanum_wheels.xacro"/>
   <xacro:include filename="base.xacro"/>

File: mobile_base_description/urdf/properties.xacro (robot description, xacro)
@@ -6,62 +6,12 @@
   <xacro:property name="chassis_height" value="0.050"/>
   <xacro:property name="chassis_mass" value="1.80"/>
-  <!-- Measured from the four wheel STL roller envelopes (millimetres on export). -->
+  <!-- Measured from the four wheel STL envelopes (millimetres on export). -->
   <xacro:property name="wheel_radius" value="0.03074443"/>
   <xacro:property name="wheel_width" value="0.03360543"/>
   <xacro:property name="wheel_mass" value="0.12"/>
-  <xacro:property name="roller_count" value="10"/>
-  <xacro:property name="roller_center_radius" value="0.02505"/>
-  <xacro:property name="roller_radius"
-                  value="${wheel_radius - roller_center_radius}"/>
-  <xacro:property name="roller_length" value="0.02580"/>
-  <xacro:property name="roller_inclination" value="${pi / 4.0}"/>
-  <xacro:property name="roller_mass" value="${wheel_mass * 0.03}"/>
-  <xacro:property name="roller_joint_damping"
-                  value="$(arg roller_joint_damping)"/>
-  <xacro:property name="roller_joint_friction"
-                  value="$(arg roller_joint_friction)"/>
-  <xacro:property name="roller_collision_model"
-                  value="$(arg roller_collision_model)"/>
-  <!--
-    husarion_cylinder emits no roller links at all, so the hub must carry the
-    whole wheel mass. The explicit-roller models leave the roller ring holding
-    its share. Total wheel mass is 0.12 kg either way.
-  -->
-  <xacro:property name="explicit_rollers"
-                  value="${roller_collision_model != 'husarion_cylinder'}"/>
-  <xacro:property name="wheel_hub_mass"
-                  value="${wheel_mass - roller_count * roller_mass
-                           if explicit_rollers else wheel_mass}"/>
-  <!--
-    Anisotropic wheel contact, used only by husarion_cylinder. A mecanum roller
-    rolls across its own axis and grips along it, so mu acts along fdir1 (the
-    roller axis) and mu2 across it. Values follow the shipping Husarion ROSbot
-    XL configuration; slip1 supplies the tangential compliance without which
-    the single-cylinder contact oscillates instead of translating.
-  -->
-  <!--
-    Driven-joint resistance. With explicit rollers the roller ring carries the
-    sliding and these values are part of the existing calibration, so they are
-    left alone. husarion_cylinder has no rollers, so every bit of joint
-    resistance runs through the wheel joint; the shipping ROSbot XL uses
-    0.001/0.001 there, against 0.05/0.01 here, and the heavier damping shows up
-    as wheel-tracking error.
-  -->
-  <xacro:property name="wheel_joint_damping"
-                  value="${0.05 if explicit_rollers else 0.001}"/>
-  <xacro:property name="wheel_joint_friction"
-                  value="${0.01 if explicit_rollers else 0.001}"/>
-  <xacro:property name="wheel_contact_mu" value="$(arg wheel_contact_mu)"/>
-  <xacro:property name="wheel_contact_mu2" value="$(arg wheel_contact_mu2)"/>
-  <xacro:property name="wheel_contact_slip1" value="$(arg wheel_contact_slip1)"/>
-  <xacro:property name="wheel_contact_slip2" value="$(arg wheel_contact_slip2)"/>
-  <!--
-    Contact friction and stiffness (mu, mu2, kp, kd) are intentionally absent
-    here. They cannot be expressed in a URDF that survives gz sdf -p, so they
-    are applied by mobile_base_bringup/scripts/generate_sim_sdf.py when the
-    simulation SDF is produced. The roller_contact_mu xacro argument is still
-    accepted so callers can pass it uniformly, but it shapes the generated
-    SDF rather than this description.
-  -->
+  <!-- Preserve the inertial radius used by the validated canonical model. -->
+  <xacro:property name="wheel_inertial_radius" value="0.02505"/>
+  <xacro:property name="wheel_joint_damping" value="0.001"/>
+  <xacro:property name="wheel_joint_friction" value="0.001"/>
   <!-- wheelbase is front-to-rear wheel-center spacing; wheel_separation is track width. -->
   <xacro:property name="wheelbase" value="0.150"/>
