Commit message: navigation cleanup and urdf change to dual layer with motors

File: mobile_base_description/urdf/base.xacro (robot description, xacro)
@@ -28,4 +28,40 @@
                           visual_xyz="-0.032786922 0.001235564 0.016969848"
                           visual_rpy="${-pi / 2.0} -0.49581568 0"/>
+    <!-- Motors share their wheel's joint origin, so the motor frame sits on
+         the output shaft it drives and the shaft runs down the wheel axis.
+         Each motor lies flat on the lower deck on one of its large gearbox
+         faces, with its shaft horizontal and pointing outboard into the wheel
+         hub, and its round can pointing inboard along the body. The mesh has
+         its shaft along the mesh Z axis, so every instance rolls +/-90 degrees
+         about X to lay that axis across the robot; front and rear differ by a
+         180 degree yaw so the can always points towards the middle of the
+         robot. Left and right are mirror images, which a rotation cannot
+         express, so the two sides rest on opposite faces. -->
+    <xacro:property name="motor_inboard_y"
+                    value="${wheel_width / 2.0 - motor_body_outer}"/>
+    <xacro:tt_gearmotor prefix="${prefix}" name="front_left"
+                        x="${wheelbase / 2.0}" y="${wheel_separation / 2.0}"
+                        z="${wheel_z}" parent="base_link"
+                        visual_xyz="${-motor_shaft_x} ${-motor_inboard_y}
+                                    ${-motor_shaft_offset}"
+                        visual_rpy="${pi / 2.0} 0 0"/>
+    <xacro:tt_gearmotor prefix="${prefix}" name="front_right"
+                        x="${wheelbase / 2.0}" y="${-wheel_separation / 2.0}"
+                        z="${wheel_z}" parent="base_link"
+                        visual_xyz="${-motor_shaft_x} ${motor_inboard_y}
+                                    ${motor_shaft_offset}"
+                        visual_rpy="${-pi / 2.0} 0 0"/>
+    <xacro:tt_gearmotor prefix="${prefix}" name="rear_right"
+                        x="${-wheelbase / 2.0}" y="${-wheel_separation / 2.0}"
+                        z="${wheel_z}" parent="base_link"
+                        visual_xyz="${motor_shaft_x} ${motor_inboard_y}
+                                    ${-motor_shaft_offset}"
+                        visual_rpy="${pi / 2.0} 0 ${pi}"/>
+    <xacro:tt_gearmotor prefix="${prefix}" name="rear_left"
+                        x="${-wheelbase / 2.0}" y="${wheel_separation / 2.0}"
+                        z="${wheel_z}" parent="base_link"
+                        visual_xyz="${motor_shaft_x} ${-motor_inboard_y}
+                                    ${motor_shaft_offset}"
+                        visual_rpy="${-pi / 2.0} 0 ${pi}"/>
   </xacro:macro>
 </robot>

File: mobile_base_description/urdf/camera.xacro (robot description, xacro)
@@ -22,5 +22,6 @@
       <parent link="${prefix}base_link"/>
       <child link="${prefix}camera_link"/>
-      <origin xyz="${chassis_length / 2.0 + camera_depth / 2.0} 0 0" rpy="0 0 0"/>
+      <origin xyz="${chassis_length / 2.0 + camera_depth / 2.0} 0 ${camera_z}"
+              rpy="0 0 0"/>
     </joint>
     <link name="${prefix}camera_optical_frame"/>

File: mobile_base_description/urdf/chassis.xacro (robot description, xacro)
@@ -1,4 +1,29 @@
 <?xml version="1.0"?>
 <robot xmlns:xacro="http://www.ros.org/wiki/xacro">
+  <!-- Shifts a ground-referenced z into base_link coordinates. -->
+  <xacro:property name="deck_z_offset" value="${-base_link_height}"/>
+  <!-- One deck plate, placed by the ground-referenced z of its bottom face. -->
+  <xacro:macro name="deck_plate" params="bottom_z thickness">
+    <visual>
+      <origin xyz="0 0 ${bottom_z + thickness / 2.0 + deck_z_offset}"
+              rpy="0 0 0"/>
+      <geometry>
+        <box size="${chassis_length} ${chassis_width} ${thickness}"/>
+      </geometry>
+      <material name="base_dark"/>
+    </visual>
+  </xacro:macro>
+  <!-- One corner standoff spanning the electronics bay. -->
+  <xacro:macro name="deck_standoff" params="x y">
+    <visual>
+      <origin
+        xyz="${x} ${y} ${lower_deck_top_z + deck_gap / 2.0 + deck_z_offset}"
+        rpy="0 0 0"/>
+      <geometry>
+        <cylinder radius="${standoff_radius}" length="${deck_gap}"/>
+      </geometry>
+      <material name="sensor_grey"/>
+    </visual>
+  </xacro:macro>
   <xacro:macro name="mobile_base_chassis" params="prefix">
     <link name="${prefix}base_footprint"/>
@@ -8,12 +33,19 @@
       <origin xyz="0 0 ${base_link_height}" rpy="0 0 0"/>
     </joint>
+    <!-- The body is a dual-deck plate frame, not a solid block: separate
+         visuals for each plate and for the corner standoffs.
+         Collision stays a single bounding box over the whole body, so the
+         planner cannot route anything through the open electronics bay. -->
     <link name="${prefix}base_link">
-      <visual>
-        <geometry>
-          <box size="${chassis_length} ${chassis_width} ${chassis_height}"/>
-        </geometry>
-        <material name="base_dark"/>
-      </visual>
+      <xacro:deck_plate bottom_z="${lower_deck_bottom_z}"
+                        thickness="${lower_deck_thickness}"/>
+      <xacro:deck_plate bottom_z="${upper_deck_bottom_z}"
+                        thickness="${upper_deck_thickness}"/>
+      <xacro:deck_standoff x="${standoff_x}" y="${standoff_y}"/>
+      <xacro:deck_standoff x="${standoff_x}" y="${-standoff_y}"/>
+      <xacro:deck_standoff x="${-standoff_x}" y="${standoff_y}"/>
+      <xacro:deck_standoff x="${-standoff_x}" y="${-standoff_y}"/>
       <collision>
+        <origin xyz="0 0 ${chassis_center_z}" rpy="0 0 0"/>
         <geometry>
           <box size="${chassis_length} ${chassis_width} ${chassis_height}"/>
@@ -22,5 +54,5 @@
       <xacro:box_inertial mass="${chassis_mass}"
                           x="${chassis_length}" y="${chassis_width}" z="${chassis_height}">
-        <origin xyz="0 0 0" rpy="0 0 0"/>
+        <origin xyz="0 0 ${chassis_center_z}" rpy="0 0 0"/>
       </xacro:box_inertial>
     </link>

File: mobile_base_description/urdf/lidar.xacro (robot description, xacro)
@@ -2,23 +2,39 @@
 <robot xmlns:xacro="http://www.ros.org/wiki/xacro">
   <xacro:macro name="mobile_base_lidar" params="prefix">
+    <!-- lidar_link is the scan plane, at mid height of the rotating head.
+         Visuals are split into the square fixed base and the cylindrical
+         rotating head so the model reads as a D500 kit; collision and inertia
+         stay one box bounding both. -->
     <link name="${prefix}lidar_link">
       <visual>
-        <origin xyz="0 0 ${-lidar_height / 2.0}" rpy="0 0 0"/>
+        <origin
+          xyz="0 0 ${-lidar_head_height / 2.0 - lidar_base_height / 2.0}"
+          rpy="0 0 0"/>
         <geometry>
-          <cylinder radius="${lidar_radius}" length="${lidar_height}"/>
+          <box size="${lidar_base_size} ${lidar_base_size}
+                     ${lidar_base_height}"/>
+        </geometry>
+        <material name="lidar_base_grey"/>
+      </visual>
+      <visual>
+        <origin xyz="0 0 0" rpy="0 0 0"/>
+        <geometry>
+          <cylinder radius="${lidar_head_radius}"
+                    length="${lidar_head_height}"/>
         </geometry>
         <material name="sensor_grey"/>
       </visual>
       <collision>
-        <origin xyz="0 0 ${-lidar_height / 2.0}" rpy="0 0 0"/>
+        <origin xyz="0 0 ${lidar_collision_z}" rpy="0 0 0"/>
         <geometry>
-          <cylinder radius="${lidar_radius}" length="${lidar_height}"/>
+          <box size="${lidar_base_size} ${lidar_base_size}
+                     ${lidar_height}"/>
         </geometry>
       </collision>
-      <xacro:cylinder_inertial mass="${lidar_mass}"
-                               radius="${lidar_radius}"
-                               length="${lidar_height}">
-        <origin xyz="0 0 ${-lidar_height / 2.0}" rpy="0 0 0"/>
-      </xacro:cylinder_inertial>
+      <xacro:box_inertial mass="${lidar_mass}"
+                          x="${lidar_base_size}" y="${lidar_base_size}"
+                          z="${lidar_height}">
+        <origin xyz="0 0 ${lidar_collision_z}" rpy="0 0 0"/>
+      </xacro:box_inertial>
     </link>
     <joint name="${prefix}base_link_to_lidar_link_joint" type="fixed">

File: mobile_base_description/urdf/materials.xacro (robot description, xacro)
@@ -16,4 +16,10 @@
     <color rgba="0.10 0.45 0.22 1.0"/>
   </material>
+  <material name="lidar_base_grey">
+    <color rgba="0.24 0.26 0.29 1.0"/>
+  </material>
+  <material name="motor_yellow">
+    <color rgba="0.92 0.85 0.15 1.0"/>
+  </material>
   <material name="sensor_grey">
     <color rgba="0.55 0.58 0.62 1.0"/>

File: mobile_base_description/urdf/mobile_base.urdf.xacro (robot description, xacro)
@@ -9,4 +9,5 @@
   <xacro:include filename="chassis.xacro"/>
   <xacro:include filename="macros/mecanum_wheels.xacro"/>
+  <xacro:include filename="macros/motors.xacro"/>
   <xacro:include filename="base.xacro"/>
   <xacro:include filename="camera.xacro"/>

File: mobile_base_description/urdf/properties.xacro (robot description, xacro)
@@ -2,8 +2,43 @@
 <robot xmlns:xacro="http://www.ros.org/wiki/xacro">
   <!-- REP-103: +X forward, +Y left, +Z up. All dimensions are SI units. -->
+  <!-- chassis_* is the body bounding box: the footprint of both deck plates
+       and the full height from lower deck underside to upper deck top. It is
+       what the single collision box and the Nav2 footprint are derived from. -->
   <xacro:property name="chassis_length" value="0.216"/>
-  <xacro:property name="chassis_width" value="0.099"/>
-  <xacro:property name="chassis_height" value="0.050"/>
+  <xacro:property name="chassis_width" value="0.100"/>
   <xacro:property name="chassis_mass" value="1.80"/>
+  <!-- Dual-deck plates. The decks are 3D-printed sheet, not a solid block, so
+       the body is modelled as visuals on base_link plus one bounding collision.
+       Deck plate thickness is set by what prints reliably in PLA. -->
+  <xacro:property name="deck_thickness" value="0.010"/>
+  <xacro:property name="lower_deck_thickness" value="${deck_thickness}"/>
+  <xacro:property name="upper_deck_thickness" value="${deck_thickness}"/>
+  <!-- Clear air between the deck facing surfaces: houses the SBC and wiring,
+       and must exceed motor_height so the motors fit under the upper deck. -->
+  <xacro:property name="deck_gap" value="0.040"/>
+  <!-- TT gearmotor, measured off the vendored mesh (mm on export). The mesh
+       frame is: X along the body (round can at X=0, gearbox at high X), Y
+       across the two large flat gearbox faces, Z along the output shaft.
+       The motor rests on a large face, so its standing height is the Y span
+       and the shaft runs horizontally into the wheel. -->
+  <xacro:property name="motor_length" value="0.0695"/>
+  <xacro:property name="motor_height" value="0.0224"/>
+  <xacro:property name="motor_span" value="0.02994"/>
+  <!-- Shaft axis position in the mesh: along the body, and above the face the
+       motor rests on. The shaft is centred in the height, so a motor sitting
+       flat puts its shaft one motor_shaft_offset above the deck. -->
+  <xacro:property name="motor_shaft_x" value="0.053"/>
+  <xacro:property name="motor_shaft_offset" value="0.0112"/>
+  <!-- Outermost body point along the shaft axis. The 8.8 mm of exposed shaft
+       outboard of it slots into the wheel hub. -->
+  <xacro:property name="motor_body_outer" value="0.00755"/>
+  <!-- Fixed-joint children are lumped into base_link by the Gazebo URDF
+       reduction, so the motors carry negligible inertia and chassis_mass
+       remains the whole-body mass of the validated motion model. -->
+  <xacro:property name="motor_mass" value="1.0e-6"/>
+  <!-- Corner standoffs between the decks. Visual only. -->
+  <xacro:property name="standoff_radius" value="0.004"/>
+  <xacro:property name="standoff_x" value="0.098"/>
+  <xacro:property name="standoff_y" value="0.042"/>
   <!-- Measured from the four wheel STL envelopes (millimetres on export). -->
   <xacro:property name="wheel_radius" value="0.03074443"/>
@@ -18,11 +53,38 @@
   <xacro:property name="wheel_separation" value="0.134"/>
   <xacro:property name="wheel_diameter" value="${2.0 * wheel_radius}"/>
-  <xacro:property name="chassis_bottom_z" value="${0.25 * wheel_diameter}"/>
-  <xacro:property name="base_link_height" value="${chassis_bottom_z + chassis_height / 2.0}"/>
+  <!-- Vertical stack, ground referenced. The motors sit on the lower deck and
+       drive the wheels directly, so the deck top is pinned one shaft offset
+       below the wheel axle. That fixes ground clearance at 9.5 mm: the wheel
+       radius is what the whole stack hangs from. -->
+  <xacro:property name="lower_deck_top_z"
+                  value="${wheel_radius - motor_shaft_offset}"/>
+  <xacro:property name="lower_deck_bottom_z"
+                  value="${lower_deck_top_z - lower_deck_thickness}"/>
+  <xacro:property name="upper_deck_bottom_z"
+                  value="${lower_deck_top_z + deck_gap}"/>
+  <xacro:property name="upper_deck_top_z"
+                  value="${upper_deck_bottom_z + upper_deck_thickness}"/>
+  <xacro:property name="chassis_height"
+                  value="${upper_deck_top_z - lower_deck_bottom_z}"/>
+  <xacro:property name="chassis_bottom_z" value="${lower_deck_bottom_z}"/>
+  <!-- base_link is pinned to the height the validated motion model was
+       identified at. The body grew upward around it, so every existing tf
+       offset, controller gain and test expectation still holds. -->
+  <xacro:property name="base_link_height" value="0.040372215"/>
   <xacro:property name="wheel_z" value="${wheel_radius - base_link_height}"/>
+  <!-- Body geometry is authored ground referenced, then shifted into
+       base_link by this offset. -->
+  <xacro:property name="chassis_center_z"
+                  value="${(lower_deck_bottom_z + upper_deck_top_z) / 2.0
+                           - base_link_height}"/>
   <xacro:property name="camera_depth" value="0.002"/>
   <xacro:property name="camera_width" value="0.010"/>
   <xacro:property name="camera_height" value="0.005"/>
   <xacro:property name="camera_mass" value="0.06"/>
+  <!-- The camera is mounted on the front face of the upper deck, centred on
+       the plate's thickness. -->
+  <xacro:property name="camera_z"
+                  value="${(upper_deck_bottom_z + upper_deck_top_z) / 2.0
+                           - base_link_height}"/>
   <xacro:property name="camera_update_rate" value="20"/>
   <xacro:property name="camera_image_width" value="640"/>
@@ -33,7 +95,17 @@
   <xacro:property name="camera_noise_mean" value="0.0"/>
   <xacro:property name="camera_noise_stddev" value="0.005"/>
-  <!-- Simulated 360-degree planar LiDAR. The link origin is the scan plane. -->
-  <xacro:property name="lidar_radius" value="0.020"/>
-  <xacro:property name="lidar_height" value="0.008"/>
+  <!-- Simulated 360-degree planar LiDAR, shaped after the D500 kit: a square
+       fixed base carrying a cylindrical rotating head. The link origin is the
+       scan plane, at mid height of the head. -->
+  <xacro:property name="lidar_base_size" value="0.048"/>
+  <xacro:property name="lidar_base_height" value="0.010"/>
+  <xacro:property name="lidar_head_radius" value="0.019"/>
+  <xacro:property name="lidar_head_height" value="0.010"/>
+  <!-- Collision and inertia use one box bounding base and head together. -->
+  <xacro:property name="lidar_height"
+                  value="${lidar_base_height + lidar_head_height}"/>
+  <!-- Centre of that bounding box, relative to the scan plane. -->
+  <xacro:property name="lidar_collision_z"
+                  value="${-lidar_base_height / 2.0}"/>
   <xacro:property name="lidar_mass" value="0.10"/>
   <xacro:property name="lidar_x" value="0.0"/>
@@ -49,16 +121,23 @@
   <xacro:property name="lidar_noise_stddev" value="0.01"/>
   <!-- Simulated IMU. Noise values are standard deviations in SI units. -->
-  <xacro:property name="imu_length" value="0.050"/>
-  <xacro:property name="imu_width" value="0.050"/>
-  <xacro:property name="imu_height" value="0.008"/>
+  <xacro:property name="imu_length" value="0.025"/>
+  <xacro:property name="imu_width" value="0.025"/>
+  <xacro:property name="imu_height" value="0.004"/>
   <xacro:property name="imu_mass" value="0.03"/>
   <xacro:property name="imu_x" value="0.0"/>
   <xacro:property name="imu_y" value="0.0"/>
-  <!-- Compact sensor stack: IMU on the chassis, LiDAR on the IMU. -->
-  <xacro:property name="chassis_top_z" value="${chassis_height / 2.0}"/>
-  <xacro:property name="imu_z" value="${chassis_top_z + imu_height / 2.0}"/>
-  <!-- lidar_link is the scan plane at the top of the LiDAR cylinder. -->
+  <!-- Sensors are placed ground referenced, then shifted into base_link.
+       chassis_top_z is the upper deck top face, the mounting surface. -->
+  <xacro:property name="chassis_top_z"
+                  value="${upper_deck_top_z - base_link_height}"/>
+  <!-- The IMU hangs under the upper deck, inside the electronics bay, where
+       it is shielded and close to the rotation centre. -->
+  <xacro:property name="imu_z"
+                  value="${upper_deck_bottom_z - imu_height / 2.0
+                           - base_link_height}"/>
+  <!-- lidar_link is the scan plane, mid height of the rotating head. -->
   <xacro:property name="lidar_z"
-                  value="${imu_z + imu_height / 2.0 + lidar_height}"/>
+                  value="${upper_deck_top_z + lidar_base_height
+                           + lidar_head_height / 2.0 - base_link_height}"/>
   <xacro:property name="imu_update_rate" value="50.0"/>
   <xacro:property name="imu_angular_velocity_noise_mean" value="0.0"/>
