Commit message: description: model the battery, motor drivers and MCU on the decks
Each link origin is the part's own centroid, so the Gazebo reduction
lumps each mass in with the right parallel-axis term.

File: mobile_base_description/urdf/base.xacro (robot description, xacro)
@@ -40,4 +40,15 @@
     <xacro:property name="motor_inboard_y"
                     value="${wheel_width / 2.0 - motor_body_outer}"/>
+    <!-- The link origin is the output shaft, which is not the centre of mass:
+         the shaft sits at motor_shaft_x along the body and is centred in the
+         motor height, so the body centroid is offset along the body and along
+         the shaft axis but not vertically. The offsets are per instance
+         because they follow the same roll and yaw as the visual: the sign of
+         the body offset flips with the 180 degree yaw between front and rear,
+         and the sign of the shaft-axis offset flips between left and right. -->
+    <xacro:property name="motor_centroid_body"
+                    value="${motor_length / 2.0 - motor_shaft_x}"/>
+    <xacro:property name="motor_centroid_axis"
+                    value="${motor_span / 2.0 + motor_inboard_y}"/>
     <xacro:tt_gearmotor prefix="${prefix}" name="front_left"
                         x="${wheelbase / 2.0}" y="${wheel_separation / 2.0}"
@@ -45,5 +56,6 @@
                         visual_xyz="${-motor_shaft_x} ${-motor_inboard_y}
                                     ${-motor_shaft_offset}"
-                        visual_rpy="${pi / 2.0} 0 0"/>
+                        visual_rpy="${pi / 2.0} 0 0"
+                        centroid_xyz="${motor_centroid_body} ${-motor_centroid_axis} 0"/>
     <xacro:tt_gearmotor prefix="${prefix}" name="front_right"
                         x="${wheelbase / 2.0}" y="${-wheel_separation / 2.0}"
@@ -51,5 +63,6 @@
                         visual_xyz="${-motor_shaft_x} ${motor_inboard_y}
                                     ${motor_shaft_offset}"
-                        visual_rpy="${-pi / 2.0} 0 0"/>
+                        visual_rpy="${-pi / 2.0} 0 0"
+                        centroid_xyz="${motor_centroid_body} ${motor_centroid_axis} 0"/>
     <xacro:tt_gearmotor prefix="${prefix}" name="rear_right"
                         x="${-wheelbase / 2.0}" y="${-wheel_separation / 2.0}"
@@ -57,5 +70,6 @@
                         visual_xyz="${motor_shaft_x} ${motor_inboard_y}
                                     ${-motor_shaft_offset}"
-                        visual_rpy="${pi / 2.0} 0 ${pi}"/>
+                        visual_rpy="${pi / 2.0} 0 ${pi}"
+                        centroid_xyz="${-motor_centroid_body} ${motor_centroid_axis} 0"/>
     <xacro:tt_gearmotor prefix="${prefix}" name="rear_left"
                         x="${-wheelbase / 2.0}" y="${wheel_separation / 2.0}"
@@ -63,5 +77,48 @@
                         visual_xyz="${motor_shaft_x} ${-motor_inboard_y}
                                     ${motor_shaft_offset}"
-                        visual_rpy="${-pi / 2.0} 0 ${pi}"/>
+                        visual_rpy="${-pi / 2.0} 0 ${pi}"
+                        centroid_xyz="${-motor_centroid_body} ${-motor_centroid_axis} 0"/>
+    <!-- Lower deck, on the centreline: the single heaviest part, kept low and
+         central so it pulls the centre of mass down rather than sideways. -->
+    <xacro:box_component prefix="${prefix}" name="battery" parent="base_link"
+                         x="${battery_x}" y="${battery_y}" z="${battery_z}"
+                         length="${battery_length}" width="${battery_width}"
+                         height="${battery_height}" mass="${battery_mass}"
+                         material="battery_grey"/>
+    <!-- Lower deck, flanking the battery. One driver per pair of motors. The
+         mesh already lies flat, so it only needs lifting by the header pin
+         drop to put its own centroid on the link origin. -->
+    <xacro:mesh_component prefix="${prefix}" name="left_motor_driver"
+                          parent="base_link"
+                          x="${driver_x}" y="${driver_y}" z="${driver_z}"
+                          length="${driver_length}" width="${driver_width}"
+                          height="${driver_height}" mass="${driver_mass}"
+                          mesh="tb6612fng.stl" material="electronics_green"
+                          visual_xyz="0 0 ${driver_mesh_offset_z}"
+                          visual_rpy="0 0 0"/>
+    <xacro:mesh_component prefix="${prefix}" name="right_motor_driver"
+                          parent="base_link"
+                          x="${driver_x}" y="${-driver_y}" z="${driver_z}"
+                          length="${driver_length}" width="${driver_width}"
+                          height="${driver_height}" mass="${driver_mass}"
+                          mesh="tb6612fng.stl" material="electronics_green"
+                          visual_xyz="0 0 ${driver_mesh_offset_z}"
+                          visual_rpy="0 0 0"/>
+    <!-- Upper deck, rear, sitting on top of the plate. The mesh stands on
+         edge with its board normal along its own +Y, so it rolls 90 degrees
+         about X to lie flat; the mesh is also authored well off its origin, so
+         the offsets carry its bounding-box centre through that same roll onto
+         the link origin. No yaw: the USB-C end is the mesh X minimum, which
+         with no yaw faces aft and stays reachable for flashing. -->
+    <xacro:mesh_component prefix="${prefix}" name="mcu" parent="base_link"
+                          x="${mcu_x}" y="${mcu_y}" z="${mcu_z}"
+                          length="${mcu_length}" width="${mcu_width}"
+                          height="${mcu_height}" mass="${mcu_mass}"
+                          mesh="esp32_s3_devkit_shield.stl"
+                          material="electronics_green"
+                          visual_xyz="${-mcu_mesh_offset_x}
+                                      ${-mcu_mesh_offset_y}
+                                      ${-mcu_mesh_offset_z}"
+                          visual_rpy="${pi / 2.0} 0 0"/>
   </xacro:macro>
 </robot>

File: mobile_base_description/urdf/macros/motors.xacro (robot description, xacro)
@@ -10,9 +10,15 @@
        own +X, so visual_xyz/visual_rpy seat the shaft on the link origin and
        point the motor can inboard - the same per-instance pose convention the
-       wheel macro uses. The motors carry negligible mass: the Gazebo URDF
-       reduction lumps fixed-joint children into base_link, and chassis_mass is
-       already the whole-body mass. -->
+       wheel macro uses.
+       The motors carry their real mass. The Gazebo URDF reduction lumps
+       fixed-joint children into base_link with parallel-axis terms, and the
+       deck plates absorb the balance so the lumped total stays at
+       total_body_mass. The inertia sits at centroid_xyz rather than at the
+       link origin, because the link origin is the output shaft: putting a
+       30 g body on the shaft instead of at its centre would misplace it by
+       nearly 30 mm. -->
   <xacro:macro name="tt_gearmotor"
-               params="prefix name parent x y z visual_xyz visual_rpy">
+               params="prefix name parent x y z visual_xyz visual_rpy
+                       centroid_xyz">
     <link name="${prefix}${name}_motor_link">
       <visual>
@@ -28,10 +34,12 @@
            and an extra collision would break the one-surface-per-wheel
            contract the Gazebo SDF generator relies on. -->
-      <inertial>
-        <origin xyz="0 0 0" rpy="0 0 0"/>
-        <mass value="${motor_mass}"/>
-        <inertia ixx="1.0e-9" ixy="0.0" ixz="0.0"
-                 iyy="1.0e-9" iyz="0.0" izz="1.0e-9"/>
-      </inertial>
+      <!-- The motor lies flat with its body along X, the shaft axis across
+           the robot, and its resting faces top and bottom, so the bounding
+           box in link axes is length by span by height. -->
+      <xacro:box_inertial mass="${motor_mass}"
+                          x="${motor_length}" y="${motor_span}"
+                          z="${motor_height}">
+        <origin xyz="${centroid_xyz}" rpy="0 0 0"/>
+      </xacro:box_inertial>
     </link>
     <joint name="${prefix}${name}_motor_joint" type="fixed">

File: mobile_base_description/urdf/materials.xacro (robot description, xacro)
@@ -22,4 +22,7 @@
     <color rgba="0.92 0.85 0.15 1.0"/>
   </material>
+  <material name="battery_grey">
+    <color rgba="0.14 0.15 0.17 1.0"/>
+  </material>
   <material name="sensor_grey">
     <color rgba="0.55 0.58 0.62 1.0"/>

File: mobile_base_description/urdf/mobile_base.urdf.xacro (robot description, xacro)
@@ -10,4 +10,5 @@
   <xacro:include filename="macros/mecanum_wheels.xacro"/>
   <xacro:include filename="macros/motors.xacro"/>
+  <xacro:include filename="macros/components.xacro"/>
   <xacro:include filename="base.xacro"/>
   <xacro:include filename="camera.xacro"/>
