Commit message: description: extend both decks into a cross and derive the mass budget

File: mobile_base_description/urdf/chassis.xacro (robot description, xacro)
@@ -3,5 +3,12 @@
   <!-- Shifts a ground-referenced z into base_link coordinates. -->
   <xacro:property name="deck_z_offset" value="${-base_link_height}"/>
-  <!-- One deck plate, placed by the ground-referenced z of its bottom face. -->
+  <!-- One deck plate, placed by the ground-referenced z of its bottom face.
+       The plate is a cross in plan view: a full-length spine at chassis_width
+       carrying the bumpers, plus a wing on each side filling the open space
+       between that side's two wheels. Three boxes rather than one, because
+       URDF has no cross primitive - and because a single box over the whole
+       envelope would swallow the wheels.
+       The wings butt against the spine edges instead of overlapping them.
+       Overlapping boxes share coplanar faces, which z-fight in RViz. -->
   <xacro:macro name="deck_plate" params="bottom_z thickness">
     <visual>
@@ -10,4 +17,19 @@
       <geometry>
         <box size="${chassis_length} ${chassis_width} ${thickness}"/>
+      </geometry>
+      <material name="base_dark"/>
+    </visual>
+    <xacro:deck_wing bottom_z="${bottom_z}" thickness="${thickness}"
+                     y="${wing_y}"/>
+    <xacro:deck_wing bottom_z="${bottom_z}" thickness="${thickness}"
+                     y="${-wing_y}"/>
+  </xacro:macro>
+  <!-- One side wing of a deck plate. -->
+  <xacro:macro name="deck_wing" params="bottom_z thickness y">
+    <visual>
+      <origin xyz="0 ${y} ${bottom_z + thickness / 2.0 + deck_z_offset}"
+              rpy="0 0 0"/>
+      <geometry>
+        <box size="${wing_length} ${wing_width} ${thickness}"/>
       </geometry>
       <material name="base_dark"/>
@@ -26,4 +48,45 @@
     </visual>
   </xacro:macro>
+  <!-- Combined inertial for the two deck plates, about their common centre. -->
+  <xacro:property name="deck_pair_separation"
+                  value="${upper_deck_bottom_z + upper_deck_thickness / 2.0
+                           - (lower_deck_bottom_z
+                              + lower_deck_thickness / 2.0)}"/>
+  <xacro:property name="deck_pair_mass" value="${2.0 * deck_mass}"/>
+  <!-- Plan-view second moments of one cross-shaped plate, summed over the
+       spine and the two wings about the plate centre. Each limb contributes
+       its own box term plus its offset from that centre. -->
+  <xacro:property name="deck_ixx_plan"
+                  value="${(chassis_length * chassis_width
+                            * chassis_width * chassis_width) / 12.0
+                           + 2.0 * (wing_length * wing_width
+                                    * (wing_width * wing_width / 12.0
+                                       + wing_y * wing_y))}"/>
+  <xacro:property name="deck_iyy_plan"
+                  value="${(chassis_width * chassis_length
+                            * chassis_length * chassis_length) / 12.0
+                           + 2.0 * (wing_width * wing_length
+                                    * wing_length * wing_length) / 12.0}"/>
+  <xacro:property name="deck_area"
+                  value="${chassis_length * chassis_width
+                           + 2.0 * wing_length * wing_width}"/>
+  <xacro:macro name="deck_pair_inertial">
+    <inertial>
+      <origin xyz="0 0 ${chassis_center_z}" rpy="0 0 0"/>
+      <mass value="${deck_pair_mass}"/>
+      <inertia
+        ixx="${deck_pair_mass * (deck_ixx_plan / deck_area
+                                 + deck_thickness * deck_thickness / 12.0
+                                 + deck_pair_separation
+                                   * deck_pair_separation / 4.0)}"
+        ixy="0.0" ixz="0.0"
+        iyy="${deck_pair_mass * (deck_iyy_plan / deck_area
+                                 + deck_thickness * deck_thickness / 12.0
+                                 + deck_pair_separation
+                                   * deck_pair_separation / 4.0)}"
+        iyz="0.0"
+        izz="${deck_pair_mass * (deck_ixx_plan + deck_iyy_plan) / deck_area}"/>
+    </inertial>
+  </xacro:macro>
   <xacro:macro name="mobile_base_chassis" params="prefix">
     <link name="${prefix}base_footprint"/>
@@ -34,7 +97,9 @@
     </joint>
     <!-- The body is a dual-deck plate frame, not a solid block: separate
-         visuals for each plate and for the corner standoffs.
-         Collision stays a single bounding box over the whole body, so the
-         planner cannot route anything through the open electronics bay. -->
+         visuals for each plate, each wing, and each corner standoff.
+         Collision follows the same cross, one box per limb, spanning the full
+         body height. The planner still cannot route through the open
+         electronics bay, but the wings' boxes stop short of the wheels in X
+         instead of a single envelope box engulfing them. -->
     <link name="${prefix}base_link">
       <xacro:deck_plate bottom_z="${lower_deck_bottom_z}"
@@ -52,8 +117,25 @@
         </geometry>
       </collision>
-      <xacro:box_inertial mass="${chassis_mass}"
-                          x="${chassis_length}" y="${chassis_width}" z="${chassis_height}">
-        <origin xyz="0 0 ${chassis_center_z}" rpy="0 0 0"/>
-      </xacro:box_inertial>
+      <collision>
+        <origin xyz="0 ${wing_y} ${chassis_center_z}" rpy="0 0 0"/>
+        <geometry>
+          <box size="${wing_length} ${wing_width} ${chassis_height}"/>
+        </geometry>
+      </collision>
+      <collision>
+        <origin xyz="0 ${-wing_y} ${chassis_center_z}" rpy="0 0 0"/>
+        <geometry>
+          <box size="${wing_length} ${wing_width} ${chassis_height}"/>
+        </geometry>
+      </collision>
+      <!-- The structural mass is the two plates, so it is carried at the
+           plates rather than at the mid-height of an imaginary solid body.
+           URDF allows one inertial per link, so the two plates are combined
+           here: equal masses at equal distances either side of their midpoint,
+           which is what a single box of their combined span and the plate
+           footprint already integrates to about the horizontal axes. The
+           parallel-axis term for the vertical separation is added explicitly,
+           since a solid box of that height would understate it. -->
+      <xacro:deck_pair_inertial/>
     </link>
   </xacro:macro>

File: mobile_base_description/urdf/properties.xacro (robot description, xacro)
@@ -5,7 +5,13 @@
        and the full height from lower deck underside to upper deck top. It is
        what the single collision box and the Nav2 footprint are derived from. -->
-  <xacro:property name="chassis_length" value="0.216"/>
+  <!-- chassis_length is the bumper-to-bumper span: the decks reach past the
+       wheels front and rear so the body takes a knock before a wheel does.
+       Ceiling is 0.250. Past that the spine corner overtakes the wheel
+       envelope as the circumscribed radius and Nav2's robot_radius (0.14 in
+       planner.yaml and local_costmap.yaml) no longer covers the body. -->
+  <xacro:property name="chassis_length" value="0.240"/>
+  <!-- Spine width. The decks also carry side wings out to the wheel outer
+       faces; chassis_overall_width below is the true widest point. -->
   <xacro:property name="chassis_width" value="0.100"/>
-  <xacro:property name="chassis_mass" value="1.80"/>
   <!-- Dual-deck plates. The decks are 3D-printed sheet, not a solid block, so
        the body is modelled as visuals on base_link plus one bounding collision.
@@ -34,7 +40,8 @@
   <xacro:property name="motor_body_outer" value="0.00755"/>
   <!-- Fixed-joint children are lumped into base_link by the Gazebo URDF
-       reduction, so the motors carry negligible inertia and chassis_mass
-       remains the whole-body mass of the validated motion model. -->
-  <xacro:property name="motor_mass" value="1.0e-6"/>
+       reduction with parallel-axis terms, so each carries its real mass and
+       the composite body inertia falls out of the reduction. The deck plates
+       absorb the balance, holding the lumped total at total_body_mass. -->
+  <xacro:property name="motor_mass" value="0.030"/>
   <!-- Corner standoffs between the decks. Visual only. -->
   <xacro:property name="standoff_radius" value="0.004"/>
@@ -53,4 +60,26 @@
   <xacro:property name="wheel_separation" value="0.134"/>
   <xacro:property name="wheel_diameter" value="${2.0 * wheel_radius}"/>
+  <!-- Deck cross section, in plan view. Each deck is a full-length spine at
+       chassis_width, plus a wing on each side filling the open space between
+       the front and rear wheel of that side. The wings butt against the spine
+       edges rather than overlapping them: coplanar faces z-fight in RViz.
+       The wings reach out to the wheel outer faces and stop short of the
+       wheels in X, so they add deck area without ever fouling a rotating
+       wheel. Every bound below is derived from the wheel geometry, so moving
+       a wheel moves the wings with it. -->
+  <xacro:property name="wheel_outer_y"
+                  value="${wheel_separation / 2.0 + wheel_width / 2.0}"/>
+  <!-- Innermost point a wheel reaches along X, at the axle height. -->
+  <xacro:property name="wheel_x_inner"
+                  value="${wheelbase / 2.0 - wheel_radius}"/>
+  <xacro:property name="wing_clearance_x" value="0.004"/>
+  <xacro:property name="wing_length"
+                  value="${2.0 * (wheel_x_inner - wing_clearance_x)}"/>
+  <xacro:property name="wing_width"
+                  value="${wheel_outer_y - chassis_width / 2.0}"/>
+  <xacro:property name="wing_y"
+                  value="${(chassis_width / 2.0 + wheel_outer_y) / 2.0}"/>
+  <!-- The widest point of the body, over the wings. -->
+  <xacro:property name="chassis_overall_width" value="${2.0 * wheel_outer_y}"/>
   <!-- Vertical stack, ground referenced. The motors sit on the lower deck and
        drive the wheels directly, so the deck top is pinned one shaft offset
@@ -78,4 +107,75 @@
                   value="${(lower_deck_bottom_z + upper_deck_top_z) / 2.0
                            - base_link_height}"/>
+  <!-- ==================== Mounted components ====================
+       The battery and the boards ride on the decks as fixed-joint children of
+       base_link. Each link origin is the part's centroid, so its inertial sits
+       at the link origin and the Gazebo URDF reduction lumps it into base_link
+       with the right parallel-axis term. Mesh-backed parts additionally carry
+       a visual pose that seats the vendored mesh on that centroid, the same
+       per-instance convention the wheel and motor macros use.
+       Deck surfaces the parts sit on, in base_link coordinates. -->
+  <xacro:property name="lower_deck_surface_z"
+                  value="${lower_deck_top_z - base_link_height}"/>
+  <xacro:property name="upper_deck_surface_z"
+                  value="${upper_deck_top_z - base_link_height}"/>
+  <!-- 2S 5200 mAh hard-case LiPo, modelled as a plain cuboid: no mesh, and
+       the case really is a rectangular block. It lies flat on the lower deck
+       on the robot centreline, low and central, which is where the single
+       heaviest part belongs. 25 mm of the 40 mm bay, leaving headroom over it.
+       The 47 mm case clears the motor bodies inboard faces by 4.3 mm. -->
+  <xacro:property name="battery_length" value="0.138"/>
+  <xacro:property name="battery_width" value="0.047"/>
+  <xacro:property name="battery_height" value="0.025"/>
+  <xacro:property name="battery_mass" value="0.250"/>
+  <xacro:property name="battery_x" value="0.0"/>
+  <xacro:property name="battery_y" value="0.0"/>
+  <xacro:property name="battery_z"
+                  value="${lower_deck_surface_z + battery_height / 2.0}"/>
+  <!-- TB6612FNG carrier, two of them, one per pair of motors. Measured off
+       the vendored mesh: the board lies in its own XY plane already, so no
+       rotation, and its header pins reach driver_pin_drop below the mesh
+       origin. Seating the pin tips on the deck puts the PCB that far above it.
+       They flank the battery in the mid-band |x| < 0.022, where no motor
+       reaches, so the 12 mm of X clearance to the motor bodies holds even
+       though the boards share the motors' Y band. -->
+  <xacro:property name="driver_length" value="0.020"/>
+  <xacro:property name="driver_width" value="0.0204"/>
+  <xacro:property name="driver_height" value="0.0117"/>
+  <xacro:property name="driver_mass" value="0.003"/>
+  <xacro:property name="driver_pin_drop" value="0.0097"/>
+  <xacro:property name="driver_x" value="0.0"/>
+  <xacro:property name="driver_y" value="0.045"/>
+  <xacro:property name="driver_z"
+                  value="${lower_deck_surface_z + driver_height / 2.0}"/>
+  <!-- Mesh centroid relative to the mesh origin, so the visual pose can put
+       that centroid on the link origin. -->
+  <xacro:property name="driver_mesh_offset_z"
+                  value="${driver_pin_drop - driver_height / 2.0}"/>
+  <!-- ESP32-S3 devkit with its shield, on top of the upper deck at the rear.
+       The USB-C end is the mesh X minimum, so with no yaw it faces aft and the
+       board can be flashed without taking the robot apart.
+       The mesh lies in its own XZ plane with the board normal along +Y, so it
+       rolls 90 degrees about X to lie flat: mesh X stays along the body, mesh
+       Z becomes the width, and the mesh Y thickness becomes the height. The
+       mesh is also authored well off its own origin, so the offsets below are
+       its bounding-box centre carried through that same roll. -->
+  <xacro:property name="mcu_length" value="0.060479"/>
+  <xacro:property name="mcu_width" value="0.025195"/>
+  <xacro:property name="mcu_height" value="0.012200"/>
+  <xacro:property name="mcu_mass" value="0.012"/>
+  <xacro:property name="mcu_x" value="-0.085"/>
+  <xacro:property name="mcu_y" value="0.0"/>
+  <xacro:property name="mcu_z"
+                  value="${upper_deck_surface_z + mcu_height / 2.0}"/>
+  <xacro:property name="mcu_mesh_offset_x" value="-0.0566490"/>
+  <xacro:property name="mcu_mesh_offset_y" value="0.0639535"/>
+  <xacro:property name="mcu_mesh_offset_z" value="0.0611090"/>
+  <!-- Reserved, deliberately empty lower-deck bays. Nothing is modelled here
+       yet, but the space is claimed so later geometry does not creep into it.
+       Front bay takes the buck converters, rear bay the main power switch and
+       the battery voltage divider. Both start outboard of where the motor
+       bodies end, so they use full deck width. -->
+  <xacro:property name="reserved_bay_inner_x" value="0.0915"/>
+  <xacro:property name="reserved_bay_outer_x" value="${chassis_length / 2.0}"/>
   <xacro:property name="camera_depth" value="0.002"/>
   <xacro:property name="camera_width" value="0.010"/>
@@ -145,3 +245,19 @@
   <xacro:property name="imu_linear_acceleration_noise_mean" value="0.0"/>
   <xacro:property name="imu_linear_acceleration_noise_stddev" value="0.02"/>
+  <!-- ==================== Mass budget ====================
+       total_body_mass is base_link's mass after the Gazebo URDF reduction has
+       lumped in every fixed-joint child. The components above carry their real
+       masses and the two deck plates absorb the balance, so the total is held
+       by construction rather than by a constant that goes stale whenever a
+       part is added. The plates are the right place for the balance: they also
+       stand in for the fasteners, wiring and the reserved power components.
+       The wheels hang off revolute joints, so they are not lumped and are not
+       counted here. -->
+  <xacro:property name="total_body_mass" value="1.80"/>
+  <xacro:property name="component_mass"
+                  value="${battery_mass + 4.0 * motor_mass
+                           + 2.0 * driver_mass + mcu_mass
+                           + lidar_mass + imu_mass + camera_mass}"/>
+  <xacro:property name="deck_mass"
+                  value="${(total_body_mass - component_mass) / 2.0}"/>
 </robot>
