Commit message: description: wrap the deck ends around the wheels and widen the footprint
The end caps run the full body width past the wheels, so an impact lands
on deck rather than on a wheel.

File: mobile_base_description/urdf/chassis.xacro (robot description, xacro)
@@ -4,35 +4,49 @@
   <xacro:property name="deck_z_offset" value="${-base_link_height}"/>
   <!-- One deck plate, placed by the ground-referenced z of its bottom face.
-       The plate is a cross in plan view: a full-length spine at chassis_width
-       carrying the bumpers, plus a wing on each side filling the open space
-       between that side's two wheels. Three boxes rather than one, because
-       URDF has no cross primitive - and because a single box over the whole
-       envelope would swallow the wheels.
-       The wings butt against the spine edges instead of overlapping them.
-       Overlapping boxes share coplanar faces, which z-fight in RViz. -->
+       The plate is the full body rectangle with the four wheel wells cut out,
+       built from five butted boxes: a central spine, an end cap at each end
+       spanning the full body width, and a side wing filling the space between
+       each side's two wheels. URDF has no such primitive, and one box over
+       the whole envelope would swallow the wheels.
+       The boxes butt rather than overlap. Overlapping boxes share coplanar
+       faces, which z-fight in RViz. -->
   <xacro:macro name="deck_plate" params="bottom_z thickness">
+    <xacro:deck_slab bottom_z="${bottom_z}" thickness="${thickness}"
+                     x="0" y="0"
+                     length="${spine_length}" width="${chassis_width}"/>
+    <xacro:deck_slab bottom_z="${bottom_z}" thickness="${thickness}"
+                     x="${cap_x}" y="0"
+                     length="${cap_length}"
+                     width="${chassis_overall_width}"/>
+    <xacro:deck_slab bottom_z="${bottom_z}" thickness="${thickness}"
+                     x="${-cap_x}" y="0"
+                     length="${cap_length}"
+                     width="${chassis_overall_width}"/>
+    <xacro:deck_slab bottom_z="${bottom_z}" thickness="${thickness}"
+                     x="0" y="${wing_y}"
+                     length="${wing_length}" width="${wing_width}"/>
+    <xacro:deck_slab bottom_z="${bottom_z}" thickness="${thickness}"
+                     x="0" y="${-wing_y}"
+                     length="${wing_length}" width="${wing_width}"/>
+  </xacro:macro>
+  <!-- One rectangular piece of a deck plate. -->
+  <xacro:macro name="deck_slab" params="bottom_z thickness x y length width">
     <visual>
-      <origin xyz="0 0 ${bottom_z + thickness / 2.0 + deck_z_offset}"
+      <origin xyz="${x} ${y} ${bottom_z + thickness / 2.0 + deck_z_offset}"
               rpy="0 0 0"/>
       <geometry>
-        <box size="${chassis_length} ${chassis_width} ${thickness}"/>
+        <box size="${length} ${width} ${thickness}"/>
       </geometry>
       <material name="base_dark"/>
     </visual>
-    <xacro:deck_wing bottom_z="${bottom_z}" thickness="${thickness}"
-                     y="${wing_y}"/>
-    <xacro:deck_wing bottom_z="${bottom_z}" thickness="${thickness}"
-                     y="${-wing_y}"/>
   </xacro:macro>
-  <!-- One side wing of a deck plate. -->
-  <xacro:macro name="deck_wing" params="bottom_z thickness y">
-    <visual>
-      <origin xyz="0 ${y} ${bottom_z + thickness / 2.0 + deck_z_offset}"
-              rpy="0 0 0"/>
+  <!-- One collision limb, spanning the full body height. -->
+  <xacro:macro name="deck_limb_collision" params="x y length width">
+    <collision>
+      <origin xyz="${x} ${y} ${chassis_center_z}" rpy="0 0 0"/>
       <geometry>
-        <box size="${wing_length} ${wing_width} ${thickness}"/>
+        <box size="${length} ${width} ${chassis_height}"/>
       </geometry>
-      <material name="base_dark"/>
-    </visual>
+    </collision>
   </xacro:macro>
   <!-- One corner standoff spanning the electronics bay. -->
@@ -54,20 +68,29 @@
                               + lower_deck_thickness / 2.0)}"/>
   <xacro:property name="deck_pair_mass" value="${2.0 * deck_mass}"/>
-  <!-- Plan-view second moments of one cross-shaped plate, summed over the
-       spine and the two wings about the plate centre. Each limb contributes
-       its own box term plus its offset from that centre. -->
+  <!-- Plan-view second moments of one deck plate about its own centre,
+       summed over the five limbs. Each limb contributes its own rectangle
+       term plus the parallel-axis term for its offset from that centre.
+       Dividing by deck_area turns these into the radii of gyration the
+       inertial below scales by mass. -->
   <xacro:property name="deck_ixx_plan"
-                  value="${(chassis_length * chassis_width
+                  value="${(spine_length * chassis_width
                             * chassis_width * chassis_width) / 12.0
+                           + 2.0 * (cap_length * chassis_overall_width
+                                    * chassis_overall_width
+                                    * chassis_overall_width) / 12.0
                            + 2.0 * (wing_length * wing_width
                                     * (wing_width * wing_width / 12.0
                                        + wing_y * wing_y))}"/>
   <xacro:property name="deck_iyy_plan"
-                  value="${(chassis_width * chassis_length
-                            * chassis_length * chassis_length) / 12.0
+                  value="${(chassis_width * spine_length
+                            * spine_length * spine_length) / 12.0
+                           + 2.0 * (cap_length * chassis_overall_width
+                                    * (cap_length * cap_length / 12.0
+                                       + cap_x * cap_x))
                            + 2.0 * (wing_width * wing_length
                                     * wing_length * wing_length) / 12.0}"/>
   <xacro:property name="deck_area"
-                  value="${chassis_length * chassis_width
+                  value="${spine_length * chassis_width
+                           + 2.0 * cap_length * chassis_overall_width
                            + 2.0 * wing_length * wing_width}"/>
   <xacro:macro name="deck_pair_inertial">
@@ -98,8 +121,8 @@
     <!-- The body is a dual-deck plate frame, not a solid block: separate
          visuals for each plate, each wing, and each corner standoff.
-         Collision follows the same cross, one box per limb, spanning the full
-         body height. The planner still cannot route through the open
-         electronics bay, but the wings' boxes stop short of the wheels in X
-         instead of a single envelope box engulfing them. -->
+         Collision follows the same outline, one box per limb, spanning the
+         full body height. The planner still cannot route through the open
+         electronics bay, but the limbs leave the four wheel wells open
+         instead of a single envelope box engulfing the wheels. -->
     <link name="${prefix}base_link">
       <xacro:deck_plate bottom_z="${lower_deck_bottom_z}"
@@ -111,22 +134,19 @@
       <xacro:deck_standoff x="${-standoff_x}" y="${standoff_y}"/>
       <xacro:deck_standoff x="${-standoff_x}" y="${-standoff_y}"/>
-      <collision>
-        <origin xyz="0 0 ${chassis_center_z}" rpy="0 0 0"/>
-        <geometry>
-          <box size="${chassis_length} ${chassis_width} ${chassis_height}"/>
-        </geometry>
-      </collision>
-      <collision>
-        <origin xyz="0 ${wing_y} ${chassis_center_z}" rpy="0 0 0"/>
-        <geometry>
-          <box size="${wing_length} ${wing_width} ${chassis_height}"/>
-        </geometry>
-      </collision>
-      <collision>
-        <origin xyz="0 ${-wing_y} ${chassis_center_z}" rpy="0 0 0"/>
-        <geometry>
-          <box size="${wing_length} ${wing_width} ${chassis_height}"/>
-        </geometry>
-      </collision>
+      <xacro:deck_limb_collision x="0" y="0"
+                                 length="${spine_length}"
+                                 width="${chassis_width}"/>
+      <xacro:deck_limb_collision x="${cap_x}" y="0"
+                                 length="${cap_length}"
+                                 width="${chassis_overall_width}"/>
+      <xacro:deck_limb_collision x="${-cap_x}" y="0"
+                                 length="${cap_length}"
+                                 width="${chassis_overall_width}"/>
+      <xacro:deck_limb_collision x="0" y="${wing_y}"
+                                 length="${wing_length}"
+                                 width="${wing_width}"/>
+      <xacro:deck_limb_collision x="0" y="${-wing_y}"
+                                 length="${wing_length}"
+                                 width="${wing_width}"/>
       <!-- The structural mass is the two plates, so it is carried at the
            plates rather than at the mid-height of an imaginary solid body.

File: mobile_base_description/urdf/properties.xacro (robot description, xacro)
@@ -6,11 +6,13 @@
        what the single collision box and the Nav2 footprint are derived from. -->
   <!-- chassis_length is the bumper-to-bumper span: the decks reach past the
-       wheels front and rear so the body takes a knock before a wheel does.
-       Ceiling is 0.250. Past that the spine corner overtakes the wheel
-       envelope as the circumscribed radius and Nav2's robot_radius (0.14 in
-       planner.yaml and local_costmap.yaml) no longer covers the body. -->
-  <xacro:property name="chassis_length" value="0.240"/>
-  <!-- Spine width. The decks also carry side wings out to the wheel outer
-       faces; chassis_overall_width below is the true widest point. -->
+       wheels front and rear so the body takes a knock before a wheel does,
+       and the end caps run the full body width so a wheel cannot be struck
+       head on. Raising it pushes the cap corner further out, which is the
+       body's circumscribed radius - Nav2's robot_radius must keep covering
+       it, so planner.yaml and local_costmap.yaml move with this value. -->
+  <xacro:property name="chassis_length" value="0.260"/>
+  <!-- Width of the central spine. The end caps and the side wings both reach
+       out to the wheel outer faces; chassis_overall_width is the real widest
+       point of the body. -->
   <xacro:property name="chassis_width" value="0.100"/>
   <!-- Dual-deck plates. The decks are 3D-printed sheet, not a solid block, so
@@ -60,12 +62,22 @@
   <xacro:property name="wheel_separation" value="0.134"/>
   <xacro:property name="wheel_diameter" value="${2.0 * wheel_radius}"/>
-  <!-- Deck cross section, in plan view. Each deck is a full-length spine at
-       chassis_width, plus a wing on each side filling the open space between
-       the front and rear wheel of that side. The wings butt against the spine
-       edges rather than overlapping them: coplanar faces z-fight in RViz.
-       The wings reach out to the wheel outer faces and stop short of the
-       wheels in X, so they add deck area without ever fouling a rotating
-       wheel. Every bound below is derived from the wheel geometry, so moving
-       a wheel moves the wings with it. -->
+  <!-- Deck outline, in plan view. Each deck is the full body rectangle with
+       the four wheel wells cut out of it, built from five butted boxes:
+           +===============================+   front cap, full body width
+           |      :                 :      |
+           |      +===+=========+===+      |   wheel wells, left and right
+           |          |  wing   |          |
+           |    spine |         |          |
+           |          |  wing   |          |
+           |      +===+=========+===+      |
+           |      :                 :      |
+           +===============================+   rear cap, full body width
+       A central spine at chassis_width running between the caps, an end cap
+       at each end spanning the full body width, and a wing on each side
+       filling the space between that side's two wheels. The five boxes butt
+       against each other rather than overlapping: coplanar faces z-fight in
+       RViz, and a box reaching into a wheel well would foul a wheel.
+       Every bound derives from the wheel geometry, so moving a wheel moves
+       the deck outline with it. -->
   <xacro:property name="wheel_outer_y"
                   value="${wheel_separation / 2.0 + wheel_width / 2.0}"/>
@@ -73,4 +85,8 @@
   <xacro:property name="wheel_x_inner"
                   value="${wheelbase / 2.0 - wheel_radius}"/>
+  <!-- Outermost point a wheel reaches along X. -->
+  <xacro:property name="wheel_x_outer"
+                  value="${wheelbase / 2.0 + wheel_radius}"/>
+  <!-- Free space left around the wheels wherever deck meets wheel well. -->
   <xacro:property name="wing_clearance_x" value="0.004"/>
   <xacro:property name="wing_length"
@@ -80,4 +96,15 @@
   <xacro:property name="wing_y"
                   value="${(chassis_width / 2.0 + wheel_outer_y) / 2.0}"/>
+  <!-- End caps. Each spans the full body width in front of, or behind, that
+       end's pair of wheels, so an impact lands on deck rather than on a wheel.
+       The cap starts one clearance outboard of the wheels and runs to the
+       bumper line, and the spine runs between the two caps. -->
+  <xacro:property name="cap_inner_x"
+                  value="${wheel_x_outer + wing_clearance_x}"/>
+  <xacro:property name="cap_length"
+                  value="${chassis_length / 2.0 - cap_inner_x}"/>
+  <xacro:property name="cap_x"
+                  value="${cap_inner_x + cap_length / 2.0}"/>
+  <xacro:property name="spine_length" value="${2.0 * cap_inner_x}"/>
   <!-- The widest point of the body, over the wings. -->
   <xacro:property name="chassis_overall_width" value="${2.0 * wheel_outer_y}"/>

Commit message: description: chamfer the bumper corners at 45 degrees from the wheel line

File: mobile_base_description/urdf/chassis.xacro (robot description, xacro)
@@ -4,37 +4,21 @@
   <xacro:property name="deck_z_offset" value="${-base_link_height}"/>
   <!-- One deck plate, placed by the ground-referenced z of its bottom face.
-       The plate is the full body rectangle with the four wheel wells cut out,
-       built from five butted boxes: a central spine, an end cap at each end
-       spanning the full body width, and a side wing filling the space between
-       each side's two wheels. URDF has no such primitive, and one box over
-       the whole envelope would swallow the wheels.
-       The boxes butt rather than overlap. Overlapping boxes share coplanar
-       faces, which z-fight in RViz. -->
+       The plate outline is the body rectangle with the four wheel wells cut
+       out and the four bumper corners chamfered at 45 degrees from the wheel
+       line. URDF has no prism primitive, so unlike the collision limbs below
+       the outline cannot be built from boxes - it is a mesh, generated from
+       these same properties by scripts/generate_deck_mesh.py and checked
+       against them by the verify_deck_mesh test so it cannot drift.
+       Both decks are identical, so one mesh serves both. It is authored
+       centred on the plate, so the visual needs no pose of its own beyond the
+       plate's height. -->
   <xacro:macro name="deck_plate" params="bottom_z thickness">
-    <xacro:deck_slab bottom_z="${bottom_z}" thickness="${thickness}"
-                     x="0" y="0"
-                     length="${spine_length}" width="${chassis_width}"/>
-    <xacro:deck_slab bottom_z="${bottom_z}" thickness="${thickness}"
-                     x="${cap_x}" y="0"
-                     length="${cap_length}"
-                     width="${chassis_overall_width}"/>
-    <xacro:deck_slab bottom_z="${bottom_z}" thickness="${thickness}"
-                     x="${-cap_x}" y="0"
-                     length="${cap_length}"
-                     width="${chassis_overall_width}"/>
-    <xacro:deck_slab bottom_z="${bottom_z}" thickness="${thickness}"
-                     x="0" y="${wing_y}"
-                     length="${wing_length}" width="${wing_width}"/>
-    <xacro:deck_slab bottom_z="${bottom_z}" thickness="${thickness}"
-                     x="0" y="${-wing_y}"
-                     length="${wing_length}" width="${wing_width}"/>
-  </xacro:macro>
-  <!-- One rectangular piece of a deck plate. -->
-  <xacro:macro name="deck_slab" params="bottom_z thickness x y length width">
     <visual>
-      <origin xyz="${x} ${y} ${bottom_z + thickness / 2.0 + deck_z_offset}"
+      <origin xyz="0 0 ${bottom_z + thickness / 2.0 + deck_z_offset}"
               rpy="0 0 0"/>
       <geometry>
-        <box size="${length} ${width} ${thickness}"/>
+        <mesh
+          filename="package://mobile_base_description/meshes/decks/deck_plate.stl"
+          scale="0.001 0.001 0.001"/>
       </geometry>
       <material name="base_dark"/>
@@ -121,8 +105,12 @@
     <!-- The body is a dual-deck plate frame, not a solid block: separate
          visuals for each plate, each wing, and each corner standoff.
-         Collision follows the same outline, one box per limb, spanning the
-         full body height. The planner still cannot route through the open
-         electronics bay, but the limbs leave the four wheel wells open
-         instead of a single envelope box engulfing the wheels. -->
+         Collision approximates that outline with one box per limb, spanning
+         the full body height. The planner still cannot route through the open
+         electronics bay, and the limbs leave the four wheel wells open
+         instead of a single envelope box engulfing the wheels. The boxes keep
+         square bumper corners where the plate is chamfered, so collision
+         over-claims two small triangles at each end: boxes are cheaper and
+         steadier in contact than a mesh, and erring outwards is the safe
+         direction for a footprint. -->
     <link name="${prefix}base_link">
       <xacro:deck_plate bottom_z="${lower_deck_bottom_z}"
