Commit message: description: close the ToF ring with four corner sensors
Eight 60 degree fans at 45 degree spacing cover the full circle with 15
degrees of overlap, on the bumper chamfers along the strafe diagonals.

File: mobile_base_description/urdf/properties.xacro (robot description, xacro)
@@ -307,4 +307,21 @@
   <xacro:property name="tof_front_x" value="${chassis_length / 2.0}"/>
   <xacro:property name="tof_side_y" value="${wheel_outer_y}"/>
+  <!-- The corner sensors sit on the 45 degree bumper chamfer, whose face runs
+       from the cap's inner corner out to the narrowed bumper edge. Its
+       midpoint is the mounting point and its outward normal is the 45 degree
+       diagonal, so these look exactly along the direction a mecanum base
+       travels when it strafes at 45 degrees - the cheapest motion it has, and
+       the one the cardinal four cannot see.
+       The chamfer is a visual-mesh feature: the deck collision boxes keep
+       square corners and over-claim these triangles. That costs nothing here
+       because gpu_lidar renders the visual scene rather than the collision
+       geometry, so the surface these apertures sit on is the surface Gazebo
+       traces against. -->
+  <xacro:property name="tof_nose_half_width"
+                  value="${wheel_outer_y - cap_length}"/>
+  <xacro:property name="tof_corner_x"
+                  value="${(cap_inner_x + chassis_length / 2.0) / 2.0}"/>
+  <xacro:property name="tof_corner_y"
+                  value="${(wheel_outer_y + tof_nose_half_width) / 2.0}"/>
   <!-- Standing on the lower deck top face, so the aperture is half a board up
        from it. The board top clears the upper deck underside by 22 mm. -->
@@ -351,5 +368,5 @@
                            + 2.0 * driver_mass + mcu_mass
                            + lidar_mass + imu_mass + camera_mass
-                           + 4.0 * tof_mass}"/>
+                           + 8.0 * tof_mass}"/>
   <xacro:property name="deck_mass"
                   value="${(total_body_mass - component_mass) / 2.0}"/>

File: mobile_base_description/urdf/tof.gazebo.xacro (robot description, xacro)
@@ -54,4 +54,8 @@
     <xacro:mobile_base_tof_gazebo_one prefix="${prefix}" name="left"/>
     <xacro:mobile_base_tof_gazebo_one prefix="${prefix}" name="right"/>
+    <xacro:mobile_base_tof_gazebo_one prefix="${prefix}" name="front_left"/>
+    <xacro:mobile_base_tof_gazebo_one prefix="${prefix}" name="front_right"/>
+    <xacro:mobile_base_tof_gazebo_one prefix="${prefix}" name="rear_left"/>
+    <xacro:mobile_base_tof_gazebo_one prefix="${prefix}" name="rear_right"/>
   </xacro:macro>
 </robot>

File: mobile_base_description/urdf/tof.xacro (robot description, xacro)
@@ -13,6 +13,6 @@
        guess.
        The component macros in macros/components.xacro cannot serve here. Both
-       pin rpy to zero on the joint, and three of these four sensors are turned
-       to face their own wall. -->
+       pin rpy to zero on the joint, and seven of these eight sensors are
+       turned to face their own wall. -->
   <xacro:macro name="mobile_base_tof" params="prefix name x y z yaw">
     <link name="${prefix}tof_${name}_link">
@@ -64,9 +64,11 @@
        point of the robot, which is the only side position whose fan clears the
        wheels - see the placement note in properties.xacro.
-       Four sensors on the cardinal axes leave 30 degree wedges on the
-       diagonals, which is where a mecanum base moves when it strafes at 45
-       degrees. Those wedges are the reason four more sensors belong on the
-       chamfered corners later; the macro above already takes an arbitrary yaw,
-       so adding them is four more calls and four more property pairs. -->
+       The four corners sit on the 45 degree bumper chamfer, looking along
+       the diagonals. Those are the directions the cardinal four cannot see,
+       and the directions a mecanum base travels when it strafes at 45
+       degrees, so they close the ring: eight fans of 60 degrees spaced 45
+       degrees apart cover the full 360 with 15 degrees of overlap at every
+       seam, and the corner apertures also sit on the part of the body that
+       reaches an obstacle first in diagonal motion. -->
   <xacro:macro name="mobile_base_tof_array" params="prefix">
     <xacro:mobile_base_tof prefix="${prefix}" name="front"
@@ -81,4 +83,16 @@
                            x="0" y="${-tof_side_y}" z="${tof_z}"
                            yaw="${-pi / 2.0}"/>
+    <xacro:mobile_base_tof prefix="${prefix}" name="front_left"
+                           x="${tof_corner_x}" y="${tof_corner_y}"
+                           z="${tof_z}" yaw="${pi / 4.0}"/>
+    <xacro:mobile_base_tof prefix="${prefix}" name="front_right"
+                           x="${tof_corner_x}" y="${-tof_corner_y}"
+                           z="${tof_z}" yaw="${-pi / 4.0}"/>
+    <xacro:mobile_base_tof prefix="${prefix}" name="rear_left"
+                           x="${-tof_corner_x}" y="${tof_corner_y}"
+                           z="${tof_z}" yaw="${3.0 * pi / 4.0}"/>
+    <xacro:mobile_base_tof prefix="${prefix}" name="rear_right"
+                           x="${-tof_corner_x}" y="${-tof_corner_y}"
+                           z="${tof_z}" yaw="${-3.0 * pi / 4.0}"/>
   </xacro:macro>
 </robot>
