Commit message: description: mount four VL53L7CX ToF sensors on the lower deck
One per body face, link origin at the optical aperture.

File: mobile_base_description/urdf/mobile_base.urdf.xacro (robot description, xacro)
@@ -15,4 +15,5 @@
   <xacro:include filename="lidar.xacro"/>
   <xacro:include filename="imu.xacro"/>
+  <xacro:include filename="tof.xacro"/>
   <xacro:include filename="mobile_base.ros2_control.xacro"/>
   <xacro:include filename="mobile_base.gazebo.xacro"/>
@@ -20,8 +21,10 @@
   <xacro:include filename="lidar.gazebo.xacro"/>
   <xacro:include filename="imu.gazebo.xacro"/>
+  <xacro:include filename="tof.gazebo.xacro"/>
   <xacro:mobile_base_assembly prefix="$(arg prefix)"/>
   <xacro:mobile_base_camera prefix="$(arg prefix)"/>
   <xacro:mobile_base_lidar prefix="$(arg prefix)"/>
   <xacro:mobile_base_imu prefix="$(arg prefix)"/>
+  <xacro:mobile_base_tof_array prefix="$(arg prefix)"/>
   <xacro:mobile_base_ros2_control
     prefix="$(arg prefix)"
@@ -33,4 +36,5 @@
     <xacro:mobile_base_lidar_gazebo prefix="$(arg prefix)"/>
     <xacro:mobile_base_imu_gazebo prefix="$(arg prefix)"/>
+    <xacro:mobile_base_tof_gazebo prefix="$(arg prefix)"/>
   </xacro:if>
 </robot>

File: mobile_base_description/urdf/properties.xacro (robot description, xacro)
@@ -247,4 +247,69 @@
   <xacro:property name="lidar_noise_mean" value="0.0"/>
   <xacro:property name="lidar_noise_stddev" value="0.01"/>
+  <!-- ==================== ToF perimeter ====================
+       Four VL53L7CX multizone Time-of-Flight sensors on the Pololu #3418
+       carrier, one at the centre of each body face. The LiDAR scan plane sits
+       at 0.0915 m and sees one horizontal slice; these sit low on the lower
+       deck and see the near field the scan plane misses, floor included.
+       The VL53L7CX is chosen over the VL53L5CX and VL53L8CX for its field of
+       view alone. With only four sensors the FoV width is what sets the size
+       of the blind wedges: 60 degrees covers 240 of 360 with 30 degree wedges
+       left on the diagonals, where the 45 degree optics of the other two parts
+       would leave 45 degree wedges. Range is the wrong thing to optimise here
+       - nothing indoors is read past a metre through a zone this coarse. -->
+  <!-- Carrier board envelope, from the Pololu #3418 product page: the stated
+       13 x 18 x 3 mm covers the populated board, regulators and level shifter
+       included, so it is what collision and inertia use. The board stands
+       upright on the lower deck with its long axis vertical, its plane
+       parallel to the body face it guards. -->
+  <xacro:property name="tof_board_thickness" value="0.003"/>
+  <xacro:property name="tof_board_width" value="0.013"/>
+  <xacro:property name="tof_board_length" value="0.018"/>
+  <xacro:property name="tof_mass" value="0.0005"/>
+  <!-- The sensor package itself, which stands proud of the board and carries
+       the aperture. The PCB slab visual takes the rest of the 3 mm, so the two
+       visuals sum to exactly the envelope above rather than overrunning it. -->
+  <xacro:property name="tof_module_length" value="0.0064"/>
+  <xacro:property name="tof_module_width" value="0.003"/>
+  <xacro:property name="tof_module_height" value="0.00175"/>
+  <xacro:property name="tof_pcb_thickness"
+                  value="${tof_board_thickness - tof_module_height}"/>
+  <!-- Optics. The part reports an 8 x 8 grid of zones over a 60 x 60 degree
+       square field of view, so each zone spans 7.5 degrees. -->
+  <xacro:property name="tof_fov" value="${radians(60)}"/>
+  <xacro:property name="tof_zones" value="8"/>
+  <xacro:property name="tof_zone_angle" value="${tof_fov / tof_zones}"/>
+  <!-- Gazebo's min_angle and max_angle are ray angles, and a ray lands at the
+       centre of its zone rather than at the edge of the field. Eight zone
+       centres across 60 degrees therefore run to 26.25 degrees, half a zone
+       inside the 30 degree FoV edge. Handing Gazebo 30 degrees would splay
+       every ray outward and quietly overstate the coverage. -->
+  <xacro:property name="tof_half_span"
+                  value="${tof_fov / 2.0 - tof_zone_angle / 2.0}"/>
+  <!-- Ranging. tof_min_range is the near dead zone: the part returns nothing
+       useful inside it, so the ray visualisation starts there rather than at
+       the aperture. -->
+  <xacro:property name="tof_min_range" value="0.02"/>
+  <xacro:property name="tof_max_range" value="3.5"/>
+  <xacro:property name="tof_range_resolution" value="0.001"/>
+  <xacro:property name="tof_update_rate" value="15.0"/>
+  <xacro:property name="tof_noise_mean" value="0.0"/>
+  <xacro:property name="tof_noise_stddev" value="0.01"/>
+  <!-- Placement. Each tof link origin is the optical aperture, the point rays
+       leave from, the same way lidar_link is the scan plane rather than the
+       body of the sensor. The aperture sits on the body's outer face and the
+       board hangs inboard behind it.
+       The side apertures sit exactly at wheel_outer_y and must stay there. The
+       wing outer face is coplanar with the wheel outer faces, so every ray in
+       the fan keeps a positive outward component and grazes past the wheel.
+       Recessing the aperture even a board thickness inboard would put the
+       outer zones of the fan into the wheel instead. -->
+  <xacro:property name="tof_front_x" value="${chassis_length / 2.0}"/>
+  <xacro:property name="tof_side_y" value="${wheel_outer_y}"/>
+  <!-- Standing on the lower deck top face, so the aperture is half a board up
+       from it. The board top clears the upper deck underside by 22 mm. -->
+  <xacro:property name="tof_z"
+                  value="${lower_deck_top_z + tof_board_length / 2.0
+                           - base_link_height}"/>
   <!-- Simulated IMU. Noise values are standard deviations in SI units. -->
   <xacro:property name="imu_length" value="0.025"/>
@@ -285,5 +350,6 @@
                   value="${battery_mass + 4.0 * motor_mass
                            + 2.0 * driver_mass + mcu_mass
-                           + lidar_mass + imu_mass + camera_mass}"/>
+                           + lidar_mass + imu_mass + camera_mass
+                           + 4.0 * tof_mass}"/>
   <xacro:property name="deck_mass"
                   value="${(total_body_mass - component_mass) / 2.0}"/>

Commit message: feat(rev-d): mount the LiDAR on the deck grid, rows 2-3 middle columns

File: mobile_base_description/urdf/mobile_base.urdf.xacro (robot description, xacro)
@@ -1,6 +1,6 @@
 <?xml version="1.0"?>
 <!-- Mecanum 01 Rev D. Sensors come back one at a time; camera.xacro,
-     lidar.xacro, tof.xacro and components.xacro are the prototype's, kept
-     here to port and not included until they are placed on the Rev D hull. -->
+     tof.xacro and components.xacro are the prototype's, kept here to port
+     and not included until they are placed on the Rev D hull. -->
 <robot name="mobile_base" xmlns:xacro="http://www.ros.org/wiki/xacro">
   <xacro:arg name="prefix" default=""/>
@@ -13,9 +13,12 @@
   <xacro:include filename="base.xacro"/>
   <xacro:include filename="imu.xacro"/>
+  <xacro:include filename="lidar.xacro"/>
   <xacro:include filename="mobile_base.ros2_control.xacro"/>
   <xacro:include filename="mobile_base.gazebo.xacro"/>
   <xacro:include filename="imu.gazebo.xacro"/>
+  <xacro:include filename="lidar.gazebo.xacro"/>
   <xacro:mobile_base_assembly prefix="$(arg prefix)"/>
   <xacro:mobile_base_imu prefix="$(arg prefix)"/>
+  <xacro:mobile_base_lidar prefix="$(arg prefix)"/>
   <xacro:mobile_base_ros2_control
     prefix="$(arg prefix)"
@@ -25,4 +28,5 @@
     <xacro:mobile_base_gazebo controllers_file="$(arg controllers_file)"/>
     <xacro:mobile_base_imu_gazebo prefix="$(arg prefix)"/>
+    <xacro:mobile_base_lidar_gazebo prefix="$(arg prefix)"/>
   </xacro:if>
 </robot>

File: mobile_base_description/urdf/properties.xacro (robot description, xacro)
@@ -30,4 +30,35 @@
   <xacro:property name="body_com_z" value="0.030"/>
   <xacro:property name="wheel_mass" value="0.08"/>
+  <!-- Deck plate top face; its M3 insert grid is 20 mm pitch, rows at
+       x = 60 .. -60 mm, columns at y = +-10 and +-30 mm. -->
+  <xacro:property name="deck_top_z" value="0.05806"/>
+  <!-- 360-degree planar LiDAR, shaped after the D500 kit: square fixed base,
+       cylindrical rotating head. Bolted on the deck grid over rows 2-3 from
+       the front and the middle two columns, holes (40, +-10) and (20, +-10)
+       mm, so its centre is x = 30 mm on the centreline. lidar_link is the
+       scan plane, mid height of the head: 73 mm, clear of the 61.3 mm hull
+       and the 60 mm wheel tops. -->
+  <xacro:property name="lidar_base_size" value="0.048"/>
+  <xacro:property name="lidar_base_height" value="0.010"/>
+  <xacro:property name="lidar_head_radius" value="0.019"/>
+  <xacro:property name="lidar_head_height" value="0.010"/>
+  <xacro:property name="lidar_height"
+                  value="${lidar_base_height + lidar_head_height}"/>
+  <xacro:property name="lidar_collision_z" value="${-lidar_base_height / 2.0}"/>
+  <xacro:property name="lidar_mass" value="0.10"/>
+  <xacro:property name="lidar_x" value="0.030"/>
+  <xacro:property name="lidar_y" value="0.0"/>
+  <xacro:property name="lidar_z"
+                  value="${deck_top_z + lidar_base_height
+                           + lidar_head_height / 2.0 - base_link_height}"/>
+  <xacro:property name="lidar_samples" value="720"/>
+  <xacro:property name="lidar_update_rate" value="10.0"/>
+  <xacro:property name="lidar_min_angle" value="${-pi}"/>
+  <xacro:property name="lidar_max_angle" value="${pi}"/>
+  <xacro:property name="lidar_min_range" value="0.10"/>
+  <xacro:property name="lidar_max_range" value="4.0"/>
+  <xacro:property name="lidar_range_resolution" value="0.01"/>
+  <xacro:property name="lidar_noise_mean" value="0.0"/>
+  <xacro:property name="lidar_noise_stddev" value="0.01"/>
   <!-- Simulated IMU, on the floor of the hull at the centre. -->
   <xacro:property name="imu_length" value="0.025"/>
